File: EAGLE/ETEST02 - Fid Cross/ETEST02.brd (EAGLE design)
At the start: 300 x 300 mm, 39 parts

Commit message: Updated corners a bit, in order to squeeze in a few more fiducials.  Exported to GERBER.  Sent to board house.
Parts:
- added FID1, FID11, FID12, FID13, FID14, FID15, FID16, FID17, FID18, FID19, FID2, FID20, FID24, FID27, FID29, FID30, FID31, FID32, FID33, FID34, FID35, FID36, FID4, FID40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: FIDUCIAL, TinWhiskers:FIDUCIAL
Other:
- outline, holes or cut-outs redrawn
