File: EAGLE/EBR01 - TMC2130 breakout board/EBR01_1.sch (EAGLE design)
At the start: 24 parts, among them J1 CPL-CON-HEADER-0.1IN-8P-M, J2 CPL-CON-HEADER-0.1IN-8P-M, J3 CPL-CON-HEADER-0.1IN-2X3P-M, Q1 CPL-REG-LIN-5V-0.1A, U1 TMC2130-LA

Commit message: Modified the BOM to reflect connector, resonator changes. All component parts for EBR01 and their equivalents on EMC03 were ordered and the BOMs were updated to reflect this. The database for the new BOM-EX extension for EAGLE was updated to include all relevant parts and debugged for future use. A preliminary choice for power connector has been made.
Parts:
- C4, C6, C7: device TinWhiskers:CPL-CAP-X7R-0603-100NF-50V -> TinWhiskers:CPL-CAP-X7R-0603-100NF-100V
Changed lines of the file:
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@@
 <layer number="2" name="Route2" color="1" fill="3" visible="no" active="no"/>
 <layer number="3" name="Route3" color="4" fill="3" visible="no" active="no"/>
+<layer number="4" name="Route4" color="1" fill="4" visible="no" active="no"/>
+<layer number="5" name="Route5" color="4" fill="4" visible="no" active="no"/>
+<layer number="6" name="Route6" color="1" fill="8" visible="no" active="no"/>
+<layer number="7" name="Route7" color="4" fill="8" visible="no" active="no"/>
+<layer number="8" name="Route8" color="1" fill="2" visible="no" active="no"/>
+<layer number="9" name="Route9" color="4" fill="2" visible="no" active="no"/>
+<layer number="10" name="Route10" color="1" fill="7" visible="no" active="no"/>
+<layer number="11" name="Route11" color="4" fill="7" visible="no" active="no"/>
+<layer number="12" name="Route12" color="1" fill="5" visible="no" active="no"/>
+<layer number="13" name="Route13" color="4" fill="5" visible="no" active="no"/>
 <layer number="14" name="Route14" color="1" fill="6" visible="no" active="no"/>
 <layer number="15" name="Route15" color="4" fill="6" visible="no" active="no"/>
@@
 <part name="GND4" library="SparkFun-Aesthetics" deviceset="GND" device=""/>
 <part name="GND5" library="SparkFun-Aesthetics" deviceset="GND" device=""/>
-<part name="C4" library="TinWhiskers" deviceset="CPL-CAP-X7R-0603-100NF-50V" device="" value="100 nF"/>
+<part name="C4" library="TinWhiskers" deviceset="CPL-CAP-X7R-0603-100NF-100V" device="" value="100 nF"/>
 <part name="C1" library="TinWhiskers" deviceset="CPL-CAP-X7R-0603-0.47UF-35V" device="" value="470 nF"/>
 <part name="GND8" library="SparkFun-Aesthetics" deviceset="GND" device=""/>
@@
 <part name="GND7" library="SparkFun-Aesthetics" deviceset="GND" device=""/>
 <part name="GND10" library="SparkFun-Aesthetics" deviceset="GND" device=""/>
-<part name="C6" library="TinWhiskers" deviceset="CPL-CAP-X7R-0603-100NF-50V" device="" value="100 nF"/>
-<part name="C7" library="TinWhiskers" deviceset="CPL-CAP-X7R-0603-100NF-50V" device="" value="100 nF"/>
+<part name="C6" library="TinWhiskers" deviceset="CPL-CAP-X7R-0603-100NF-100V" device="" value="100 nF"/>
+<part name="C7" library="TinWhiskers" deviceset="CPL-CAP-X7R-0603-100NF-100V" device="" value="100 nF"/>
 <part name="GND11" library="SparkFun-Aesthetics" deviceset="GND" device=""/>
 <part name="GND12" library="SparkFun-Aesthetics" deviceset="GND" device=""/>
@@
 <instance part="GND4" gate="1" x="172.72" y="88.9"/>
 <instance part="GND5" gate="1" x="147.32" y="88.9"/>
-<instance part="C4" gate="C1" x="210.82" y="172.72" smashed="yes">
+<instance part="C4" gate="G$1" x="210.82" y="172.72" smashed="yes">
 <attribute name="NAME" x="211.328" y="173.355" size="1.778" layer="95"/>
 <attribute name="VALUE" x="210.566" y="170.307" size="1.778" layer="96"/>
@@
 <instance part="GND7" gate="1" x="223.52" y="88.9"/>
 <instance part="GND10" gate="1" x="236.22" y="88.9"/>
-<instance part="C6" gate="C1" x="259.08" y="170.18" smashed="yes" rot="R270">
+<instance part="C6" gate="G$1" x="259.08" y="170.18" smashed="yes" rot="R270">
 <attribute name="NAME" x="259.842" y="173.355" size="1.778" layer="95"/>
 <attribute name="VALUE" x="259.334" y="168.275" size="1.778" layer="96"/>
 </instance>
-<instance part="C7" gate="C1" x="271.78" y="170.18" smashed="yes" rot="R270">
+<instance part="C7" gate="G$1" x="271.78" y="170.18" smashed="yes" rot="R270">
 <attribute name="NAME" x="272.542" y="173.101" size="1.778" layer="95"/>
 <attribute name="VALUE" x="272.288" y="168.529" size="1.778" layer="96"/>
@@
 <wire x1="271.78" y1="180.34" x2="259.08" y2="180.34" width="0.6096" layer="91"/>
 <wire x1="259.08" y1="180.34" x2="256.54" y2="180.34" width="0.6096" layer="91"/>
-<pinref part="C4" gate="C1" pin="2"/>
+<pinref part="C4" gate="G$1" pin="2"/>
 <wire x1="213.36" y1="172.72" x2="256.54" y2="172.72" width="0.1524" layer="91"/>
 <wire x1="256.54" y1="172.72" x2="256.54" y2="180.34" width="0.1524" layer="91"/>
-<pinref part="C6" gate="C1" pin="1"/>
+<pinref part="C6" gate="G$1" pin="1"/>
 <wire x1="259.08" y1="175.26" x2="259.08" y2="180.34" width="0.6096" layer="91"/>
-<pinref part="C7" gate="C1" pin="1"/>
+<pinref part="C7" gate="G$1" pin="1"/>
 <wire x1="271.78" y1="175.26" x2="271.78" y2="180.34" width="0.6096" layer="91"/>
 <junction x="259.08" y="180.34"/>
@@
 </segment>
 <segment>
-<pinref part="C6" gate="C1" pin="2"/>
+<pinref part="C6" gate="G$1" pin="2"/>
 <pinref part="GND12" gate="1" pin="GND"/>
 <wire x1="259.08" y1="167.64" x2="259.08" y2="165.1" width="0.6096" layer="91"/>
 </segment>
 <segment>
-<pinref part="C7" gate="C1" pin="2"/>
+<pinref part="C7" gate="G$1" pin="2"/>
 <pinref part="GND11" gate="1" pin="GND"/>
 <wire x1="271.78" y1="167.64" x2="271.78" y2="165.1" width="0.6096" layer="91"/>
@@
 <segment>
 <pinref part="U1" gate="G$1" pin="VCP"/>
-<pinref part="C4" gate="C1" pin="1"/>
+<pinref part="C4" gate="G$1" pin="1"/>
 <wire x1="203.2" y1="175.26" x2="205.74" y2="175.26" width="0.1524" layer="91"/>
 <wire x1="205.74" y1="175.26" x2="205.74" y2="172.72" width="0.1524" layer="91"/>
