File: EAGLE/EMC03 - Motion Control/EMC03-Motion Control.brd (EAGLE design)
At the start: 150 x 129.9 mm, 153 parts, among them IC1 74ACT244DW, IC2 74ACT244DW, J1 CONN-0.1-S-1X3, J10 UART0, J11 HR911105A, J12 USD-SOCKETSMD, J13 USB-B, J14 SWD, J17 CONN-0.1-S-1X3, J18 CONN-0.1-S-2X3, J19 CONN-0.1-S-2X3, J2 CONN-0.1-S-1X3, J20 CONN-0.1-S-2X3, J22A OSTTH050160, J3 CONN-0.1-S-1X3, J31 CONN-0.1-S-1X2, J4 CONN-0.1-RA-1X4, J4A MOT-X, J5 CONN-0.1-RA-1X4, J5A MOT-Y, J6 CONN-0.1-RA-1X4, J6A MOT-Z, J7 CONN-0.1-RA-1X3, J7A CONN-RECT-3PINJST_PH_2MM, J8 CONN-0.1-RA-1X3, J8A CONN-RECT-3PINJST_PH_2MM, J9 CONN-0.1-RA-1X3, J9A CONN-RECT-3PINJST_PH_2MM, Q1 25MHz, U1 LPC1768, U2 SP3485, U3 CPL-ETH-PHY-LAN8720A, U4 74LVC1G04, U5 TC1015-3.3VCT713

Commit message: Integrated motor drivers into the EMC03 schematic, E-checked the EBR01 board with the netlist. Began similarifying things cromulently.
Parts:
- removed J20: CONN-0.1-S-2X3, !con-lstb:MA03-2
- removed J4A: MOT-X, FirePick:CONN-JST-PH_2.0MM_4PIN-SMT-RA
- removed J5A: MOT-Y, FirePick:CONN-JST-PH_2.0MM_4PIN-SMT-RA
- removed J6: CONN-0.1-RA-1X4, !con-lstb:MA04-1
- removed J6A: MOT-Z, FirePick:CONN-JST-PH_2.0MM_4PIN-SMT-RA
- removed S1: (no value), SparkFun:TACTILE_SWITCH_SMD
- removed STEPSTICK1, STEPSTICK2, STEPSTICK3: STEPSTICK, FirePick:STEPSTICK
- added C37: 220uF, TinWhiskers:C-SMD-10MM
- added C38: 470uF, TinWhiskers:C-SMD-10MM
- added C39, C41, C42, C51, C52, C61, C62, C64, C65, C74: 100 nF, TinWhiskers:C0603
- added C40, C63: 470 nF, TinWhiskers:C0603
- added C43, C44, C45, C46, C53, C54, C55, C56, C66, C67, C68, C69: 470pF, TinWhiskers:C0603
- added C47, C48, C57, C58, C70, C71: 100nF, TinWhiskers:C0603
- added C49, C59, C72: 22 nF, TinWhiskers:C0603
- added C50, C60, C73: 0.33uF, TinWhiskers:C0603
- added D10, D11, D12, D13, D14, D3, D4, D5, D6, D7, D8, D9: MSS1P6, TinWhiskers:MICRO-SMP
- added D2: SJPB-H6, TinWhiskers:DIO-SM2
- added J15, J16: CPL-CON-HEADER-0.1IN-8P-M, TinWhiskers:CON-HDR-8POS-MALE
- added L1: 100uH, TinWhiskers:L-SMD-12.5MM
- added LOGO10, LOGO11, LOGO12: LOGO-FIREPICKLARGE, FirePick:LOGO-FIREPICK
- added LOGO9: LOGO-CC-BY-SALARGE, FirePick:LOGO-CC-BY-SA
- added Q2, Q3, Q4: CPL-REG-LIN-5V-0.1A, TinWhiskers:SOT-89
- added R43: 1.2K, TinWhiskers:R0603
- added R44: 10K, TinWhiskers:R0603
- added R45, R46, R47: 0.22, TinWhiskers:R1206
- added U6: SI-8050JD, TinWhiskers:TO263-5
- added U7, U8, U9: TMC2130-LA, TinWhiskers:QFN36-(5X6)
- C15, C17: value 100uF -> 100 nF; device rcl:PANASONIC_D -> TinWhiskers:C0603
- C16: value 100uF -> 470 nF; device rcl:PANASONIC_D -> TinWhiskers:C0603
- J18, J19: value CONN-0.1-S-2X3 -> CPL-CON-HEADER-0.1IN-8P-M; device !con-lstb:MA03-2 -> TinWhiskers:CON-HDR-8POS-MALE
- J4, J5: value CONN-0.1-RA-1X4 -> CPL-CON-HEADER-0.1IN-8P-M; device !con-lstb:MA04-1 -> TinWhiskers:CON-HDR-8POS-MALE
- R1, R6, R7: value 100K -> 0.22; device SparkFun-Resistors:0805 -> TinWhiskers:R1206
- R42: value 1K -> 470R
- moved R7 1047.7 mm to (129.9, 1104.2), turned to 0 degrees
- moved LED10 993.6 mm to (-65.0, -1428.9)
- moved LED9 965.6 mm to (-65.0, -1364.0)
- moved J19 804.0 mm to (129.9, 844.4), turned to 0 degrees
- moved R6 736.5 mm to (129.9, 779.4), turned to 0 degrees
- moved J18 736.0 mm to (65.0, 844.4)
- moved R1 671.0 mm to (65.0, 779.4), turned to 0 degrees
- moved C17 616.7 mm to (0.00, 649.5), turned to 0 degrees
- moved C16 605.5 mm to (-65.0, 649.5), turned to 0 degrees
- moved J5 502.9 mm to (129.9, 519.6), turned to 0 degrees
- moved C15 489.6 mm to (194.9, 584.6), turned to 0 degrees
- moved J4 393.2 mm to (65.0, 519.6), turned to 0 degrees
Connections:
- net VRIN renamed VR_IN
- removed net !RESET: S1.3, S1.4
- removed net N$11: STEPSTICK1.!RESET!, STEPSTICK1.!SLEEP!
- removed net N$16: STEPSTICK2.!RESET!, STEPSTICK2.!SLEEP!
- removed net N$24: STEPSTICK3.!RESET!, STEPSTICK3.!SLEEP!
- removed net SD_MISO: J12.7, R37.2, U1.77
- removed net SD_MOSI: J12.3, R36.2, U1.76
- removed net SD_SCK: J12.5, U1.78
- removed net VROUT: C36.2, U5.5
- removed net X1A: J4.2, J4A.2, STEPSTICK1.1A
- removed net X1B: J4.1, J4A.1, STEPSTICK1.1B
- removed net X2A: J4.3, J4A.3, STEPSTICK1.2A
- removed net X2B: J4.4, J4A.4, STEPSTICK1.2B
- removed net X_DIR: STEPSTICK1.DIR
- removed net X_MS1: J18.1, R1.2, STEPSTICK1.MS1
- removed net X_MS2: J18.3, STEPSTICK1.MS2
- removed net X_MS3: J18.5, STEPSTICK1.MS3
- removed net X_STEP: STEPSTICK1.STEP
- removed net Y1A: J5.2, J5A.2, STEPSTICK2.1A
- removed net Y1B: J5.1, J5A.1, STEPSTICK2.1B
- removed net Y2A: J5.3, J5A.3, STEPSTICK2.2A
- removed net Y2B: J5.4, J5A.4, STEPSTICK2.2B
- removed net Y_DIR: STEPSTICK2.DIR
- removed net Y_MS1: J19.1, R6.2, STEPSTICK2.MS1
- removed net Y_MS2: J19.3, STEPSTICK2.MS2
- removed net Y_MS3: J19.5, STEPSTICK2.MS3
- removed net Y_STEP: STEPSTICK2.STEP
- removed net Z1A: J6.2, J6A.2, STEPSTICK3.1A
- removed net Z1B: J6.1, J6A.1, STEPSTICK3.1B
- removed net Z2A: J6.3, J6A.3, STEPSTICK3.2A
- removed net Z2B: J6.4, J6A.4, STEPSTICK3.2B
- removed net Z_DIR: STEPSTICK3.DIR
- removed net Z_MS1: J20.1, R7.2, STEPSTICK3.MS1
- removed net Z_MS2: J20.3, STEPSTICK3.MS2
- removed net Z_MS3: J20.5, STEPSTICK3.MS3
- removed net Z_STEP: STEPSTICK3.STEP
- new net !ENABLE!: J16.1, J19.1, J5.1, U7.22, U8.22, U9.22
- new net !RESET!: J16.5
- new net !SLEEP!: J16.6
- new net +24V: C15.2, C16.2, C17.1, C39.2, C40.2, C41.1, C42.1, C50.2, C52.1, C60.2, C62.2, C63.2, C64.1, C65.1, C73.2, Q2.1, Q3.1, Q4.1, R44.2, U7.16, U7.30, U7.31, U8.16, U8.30, U8.31, U9.16, U9.30, U9.31
- new net 1A_1: C45.1, D5.NEG, J15.5, U7.32
- new net 1A_2: C68.1, D13.NEG, J18.5, U9.32
- new net 1A_3: C55.1, D9.NEG, J4.5, U8.32
- new net 1B_1: C46.1, D6.NEG, J15.6, U7.34
- new net 1B_2: C69.1, D14.NEG, J18.6, U9.34
- new net 1B_3: C56.1, D10.NEG, J4.6, U8.34
- new net 2A_1: C44.1, D4.NEG, J15.4, U7.13
- new net 2A_2: C67.1, D12.NEG, J18.4, U9.13
- new net 2A_3: C54.1, D8.NEG, J4.4, U8.13
- new net 2B_1: C43.1, D3.NEG, J15.3, U7.15
- new net 2B_2: C66.1, D11.NEG, J18.3, U9.15
- new net 2B_3: C53.1, D7.NEG, J4.3, U8.15
- new net BRA: C48.1, D3.POS, D4.POS, R45.2, U7.33
- new net BRA2: C71.1, D11.POS, D12.POS, R7.2, U9.33
- new net BRA3: C58.1, D7.POS, D8.POS, R1.2, U8.33
- new net BRB: C47.1, D5.POS, D6.POS, R46.2, U7.14
- new net BRB2: C70.1, D13.POS, D14.POS, R47.2, U9.14
- new net BRB3: C57.1, D10.POS, D9.POS, R6.2, U8.14
- new net CLK: U7.1, U8.1, U9.1
- new net CPI: C49.2, U7.28
- new net CPI1: C59.2, U8.28
- new net CPI2: C72.2, U9.28
- new net CPO: C49.1, U7.27
- new net CPO1: C59.1, U8.27
- new net CPO2: C72.1, U9.27
- new net DIR: J16.8, J19.8, J5.8, U7.7, U8.7, U9.7
- new net MISO: J12.7, R37.2, U1.77, U7.5, U8.5, U9.5
- new net MOSI: J12.3, R36.2, U1.76, U7.4, U8.4, U9.4
- new net MS1: J16.2
- new net MS2: J16.3
- new net MS3: J16.4
- new net N$10: LED9.A, R43.1
- new net N$12: LED10.A, R44.1
- new net N$14: D2.POS, L1.P$1, U6.2
- new net SCK: J12.5, U1.78, U7.3, U8.3, U9.3
- new net SPI_!CS1: U1.9, U7.2
- new net SPI_!CS2: U1.8, U9.2
- new net SPI_!CS3: U1.7, U8.2
- new net STEP: J16.7, J19.7, J5.7, U7.6, U8.6, U9.6
- new net VCC1: C51.2, Q2.3, U7.26, U7.8
- new net VCC2: C74.2, Q4.3, U9.26, U9.8
- new net VCC3: C61.2, Q3.3, U8.26, U8.8
- new net VCP: C39.1, U7.29
- new net VCP1: C15.1, U8.29
- new net VCP2: C62.1, U9.29
- new net VSW_IN: C37.POS, U6.1
- net !X_ENABLE: no longer STEPSTICK1.!ENABLE!
- net !Y_ENABLE: no longer STEPSTICK2.!ENABLE!
- net !Z_ENABLE: no longer STEPSTICK3.!ENABLE!
- net +3V3: now also C10.2, C36.2, C5.2, C6.2, C7.2, C8.2, C9.2, FB2.2, R42.2, U1.28, U1.42, U1.54, U1.71, U1.84, U1.96, U5.5
- net +5V: now also C38.POS, L1.P$2, R43.2, U6.4; no longer J18.2, J18.4, J18.6, J19.2, J19.4, J19.6, J20.2, J20.4, J20.6, STEPSTICK1.VDD, STEPSTICK2.VDD, STEPSTICK3.VDD
- net 12V: no longer C15.+, C16.+, C17.+, STEPSTICK1.VMOT, STEPSTICK2.VMOT, STEPSTICK3.VMOT
- net GND: now also C16.1, C17.2, C37.NEG, C38.NEG, C40.1, C41.2, C42.2, C43.2, C44.2, C45.2, C46.2, C47.2, C48.2, C50.1, C51.1, C52.2, C53.2, C54.2, C55.2, C56.2, C57.2, C58.2, C60.1, C61.1, C63.1, C64.2, C65.2, C66.2, C67.2, C68.2, C69.2, C70.2, C71.2, C73.1, C74.1, D2.NEG, J15.2, J15.8, J18.2, J18.8, J4.2, J4.8, LED10.C, LED8.C, LED9.C, Q2.2, Q3.2, Q4.2, R45.1, R46.1, R47.1, U6.3, U6.5, U6.GND, U7.12, U7.18, U7.24, U7.35, U7.36, U7.PAD, U8.12, U8.18, U8.24, U8.35, U8.36, U8.PAD, U9.12, U9.18, U9.24, U9.35, U9.36, U9.PAD; no longer C15.-, C16.-, C17.-, LED4.C, S1.1, S1.2, STEPSTICK1.GND, STEPSTICK1.GND@2, STEPSTICK2.GND, STEPSTICK2.GND@2, STEPSTICK3.GND, STEPSTICK3.GND@2
- net N$9: now also LED8.A; no longer LED4.A
- net VDD: now also J15.7, J18.7, J4.7; no longer C10.2, C5.2, C6.2, C7.2, C8.2, C9.2, FB2.2, R42.2, U1.28, U1.42, U1.54, U1.71, U1.84, U1.96
Routing:
- net 12V: track 323.5 -> 23.4 mm, vias 3 -> 0
- net +5V: track 490.6 -> 371.8 mm
- net !RESET: track 88.9 -> 0.00 mm, vias 4 -> 0
- net X2B: track 37.9 -> 0.00 mm
- net X1A: track 37.6 -> 0.00 mm
- net X1B: track 36.5 -> 0.00 mm
- net X2A: track 35.8 -> 0.00 mm
- net Y2B: track 24.6 -> 0.00 mm
- net Y1B: track 24.1 -> 0.00 mm
- net Y2A: track 22.8 -> 0.00 mm
- net Y1A: track 22.7 -> 0.00 mm
- net Z2B: track 20.0 -> 0.00 mm
- net Z1B: track 19.9 -> 0.00 mm
- net Z1A: track 18.2 -> 0.00 mm
- net Z2A: track 18.2 -> 0.00 mm
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
Commit message: Integrated the MCU into the EMC02 schematic. The EMC03 schematic is accompanied by a BOM and pinout for the LPC1768. The pinout does not yet reflect the changes of 9/11/15, but all the major connections are accurate (power, MicroSD, RS-485, USB-B). The nomenclature on the Ethernet connections has changed slightly due to more accuracy on the schematic with regards to the reference designators, part numbers, etc. A few parts in the Tin Whiskers library were discovered to have minor aesthetic errors which were corrected. The existing devices from the legacy board which weren't located in an accessible library were replaced with equivalent (or in the case of resistors and caps, smaller) packages to facilitate routing and board layout. The schematic will be finished pending a design decision made with regards to the RS-485 connector, PWR input connector, and main clock oscillator for the MCU. Shit.
Parts:
- removed IC1, IC2: 74ACT244DW, 74xx-eu:SO20W
- removed J16, J18, J19: CPL-CON-HEADER-0.1IN-8P-M, TinWhiskers:CON-HDR-8POS-MALE
- removed J17: CONN-0.1-S-1X3, !con-lstb:MA03-1
- removed J22A: OSTTH050160, FirePick:CONN-OSTTH050160
- removed J31: CONN-0.1-S-1X2, !con-lstb:MA02-1
- removed J7A, J8A, J9A: CONN-RECT-3PINJST_PH_2MM, FirePick:CONN-JST_PH-2.0MM-3PIN-SMT-RA
- removed LED10, LED8, LED9: RED, TinWhiskers:LED0603
- removed Q3, Q4: CPL-REG-LIN-5V-0.1A, TinWhiskers:SOT-89
- removed S4: 147873-2, TinWhiskers:0603
- removed U9: TMC2130-LA, TinWhiskers:QFN36-(5X6)
- added C75: 12pF, TinWhiskers:C0603
- added J6: CONN-0.1-RA-1X3, TinWhiskers:CON-HDR-3POS-MALE
- added RJ2: HR911105A, TinWhiskers:MAGJACK(HR911105A)
- added S1: SWS001, smd-special:SMS-001
- added VR1: TC1015-3.3VCT713, TinWhiskers:SOT-23-5
- added VR2: SI-8050JD, TinWhiskers:TO263-5
- added VR3, VR4, VR5: KA78L05AMTF, TinWhiskers:SOT-89
- C1: value 0.1u -> 12pF; device SparkFun-Capacitors:0805 -> TinWhiskers:C0603
- C2, C4: value 0.1u -> 0.1uF
- J1: value CONN-0.1-S-1X3 -> UART0; device !con-lstb:MA03-1 -> TinWhiskers:CON-HDR-6POS-MALE
- J10: value UART0 -> CPL-CON-HEADER-0.1IN-8P-M; device TinWhiskers:CON-HDR-6POS-MALE -> TinWhiskers:CON-HDR-8POS-MALE
- J11: value HR911105A -> 8-PIN HDR; device TinWhiskers:MAGJACK(HR911105A) -> TinWhiskers:CON-HDR-8POS-MALE
- J12: value USD-SOCKETSMD -> 8-PIN HDR; device TinWhiskers:MICRO-SD-SOCKET-PP -> TinWhiskers:CON-HDR-8POS-MALE
- J13: value USB-B -> 8-PIN HDR; device TinWhiskers:USB-B(THRU) -> TinWhiskers:CON-HDR-8POS-MALE
- J14: value SWD -> 8-PIN HDR; device TinWhiskers:FTSH-105-01-XXX-DV-K -> TinWhiskers:CON-HDR-8POS-MALE
- J15: value CPL-CON-HEADER-0.1IN-8P-M -> 8-PIN HDR
- J2: value CONN-0.1-S-1X3 -> SWD; device !con-lstb:MA03-1 -> TinWhiskers:FTSH-105-01-XXX-DV-K
- J3: value CONN-0.1-S-1X3 -> USB-B; device !con-lstb:MA03-1 -> TinWhiskers:USB-B(THRU)
- J4: value CPL-CON-HEADER-0.1IN-8P-M -> USD-SOCKETSMD; device TinWhiskers:CON-HDR-8POS-MALE -> TinWhiskers:MICRO-SD-SOCKET-PP
- J5: value CPL-CON-HEADER-0.1IN-8P-M -> CONN-0.1-RA-1X3; device TinWhiskers:CON-HDR-8POS-MALE -> TinWhiskers:CON-HDR-3POS-MALE
- J7: device !con-lstb:MA03-1 -> TinWhiskers:CON-HDR-3POS-MALE
- J8: value CONN-0.1-RA-1X3 -> OSTTH050160; device !con-lstb:MA03-1 -> TinWhiskers:CON-HDR-6POS-MALE
- J9: value CONN-0.1-RA-1X3 -> CONN-0.1-S-1X2; device !con-lstb:MA03-1 -> TinWhiskers:CON-HDR-2POS-MALE
- LED1, LED2, LED3: value AMBER -> GREEN; device SparkFun-LED:LED-1206-NO_SILK -> TinWhiskers:LED0603
- LED5, LED6, LED7: value GREEN -> RED
- Q1: value 25MHz -> TBD
- Q2: value CPL-REG-LIN-5V-0.1A -> 25MHz; device TinWhiskers:SOT-89 -> TinWhiskers:HC-49/U-S
- R17: value 20K -> 10K; device SparkFun-Resistors:0805 -> TinWhiskers:R0603
- R18, R36: value 10K -> 10k
- R19: value 10k -> 20K; device TinWhiskers:R0603 -> SparkFun-Resistors:0805
- R2: value 10K -> 0.22; device SparkFun-Resistors:0805 -> TinWhiskers:R1206
- R23, R24, R37: value 10k -> 10K
- R25, R26: device SparkFun-Resistors:0805 -> TinWhiskers:R0603
- R27: value 10K -> 100K
- R28: value 4.7K -> 10K; device SparkFun-Resistors:0805 -> TinWhiskers:R0603
- R29: value 100K -> 4.7K
- R3: value 1k -> 1M; device SparkFun-Resistors:0805 -> TinWhiskers:R0603
- R33: value 10K -> 330R
- R35: value 330R -> 10K
- R38: value 10K -> 1K
- R4, R5: value 1k -> 10k; device SparkFun-Resistors:0805 -> TinWhiskers:R0603
- R40: value 1K -> 100R
- R41: value 100R -> 470R
- R42: value 470R -> 1.2K
- R43: value 1.2K -> 10K
- R44: value 10K -> 0.22; device TinWhiskers:R0603 -> TinWhiskers:R1206
- R6, R7: value 0.22 -> 470R; device TinWhiskers:R1206 -> TinWhiskers:R0603
- R8, R9: value 10K -> 470R; device SparkFun-Resistors:0805 -> TinWhiskers:R0603
- S2: value SWS001 -> 147873-2; device smd-special:SMS-001 -> TinWhiskers:0603
- TP2: value +12V -> +5V
- TP3: value GND -> +24V
- TP4: value +5V -> GND
- U5: value TC1015-3.3VCT713 -> 74AHCT; device TinWhiskers:SOT-23-5 -> TinWhiskers:SC70
- U6: value SI-8050JD -> TMC2130-LA; device TinWhiskers:TO263-5 -> TinWhiskers:QFN36-(5X6)
- moved R44 2017.7 mm to (65.0, 454.7)
- moved Q1 1394.6 mm to (-454.7, 454.7)
- moved LOGO9 1388.5 mm to (-324.8, -259.8)
- moved R43 1324.8 mm to (-324.8, -194.9)
- moved R7 1313.6 mm to (-65.0, -194.9)
- moved U6 1305.5 mm to (194.9, 194.9)
- moved J14 1276.1 mm to (129.9, 519.6)
- moved R6 1194.1 mm to (-324.8, -324.8)
- moved R33 1104.2 mm to (584.6, 259.8)
- moved C37 1047.3 mm to (-65.0, -129.9)
- moved C38 1047.3 mm to (-194.9, -259.8)
- moved D2 1047.3 mm to (-194.9, -194.9)
- moved L1 1047.3 mm to (-194.9, -129.9)
- moved R40 1027.0 mm to (714.5, 259.8)
- moved LOGO10 1016.7 mm to (-519.6, 259.8)
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- renumbered TP5 to TP1
Connections:
- net N$1 renamed RXD0PIN
- net N$18 renamed RXD1PIN
- net N$19 renamed CRSPIN
- net N$2 renamed DPWR
- removed net !ENABLE!: J16.1, J19.1, J5.1, U7.22, U8.22, U9.22
- removed net !X_ENABLE: IC1.18, R2.1
- removed net !X_ENABLE_BUF: IC1.2
- removed net !Y_ENABLE: IC1.16, R8.1
- removed net !Y_ENABLE_BUF: IC1.4
- removed net !Z_ENABLE: IC1.14, R9.1
- removed net !Z_ENABLE_BUF: IC1.6
- removed net 12V: TP2.1
- removed net 3.3V: TP1.1
- removed net AVR_RXD: LED3.C
- removed net AVR_TXD: LED2.C
- removed net D13_LED: LED1.C
- removed net DIR: J16.8, J19.8, J5.8, U7.7, U8.7, U9.7
- removed net GND1: C27.1
- removed net IOREF: R29.2
- removed net N$21: LED2.A, R4.2
- removed net N$22: LED3.A, R5.2
- removed net N$4: LED1.A, R3.1
- removed net RXI: J10.5
- removed net SERVO1: IC1.9, J1.1
- removed net SERVO1_BUF: IC1.11
- removed net SERVO2: IC1.7, J2.1
- removed net SERVO2_BUF: IC1.13
- removed net SERVO3: IC1.5, J3.1
- removed net SERVO3_BUF: IC1.15
- removed net SERVO4: IC1.3, J17.1
- removed net SERVO4_BUF: IC1.17
- removed net STEP: J16.7, J19.7, J5.7, U7.6, U8.6, U9.6
- removed net TXO: J10.4
- removed net VDD: J15.7, J18.7, J4.7
- removed net X_MIN_PIN: R21.2, R25.1
- removed net Y_MIN_PIN: R20.2, R26.1
- removed net Z_MIN_PIN: R17.2, R27.1
- new net !ENABLE: J10.1, J12.1, J14.1, R28.1, U6.22, U7.22, U8.22
- new net !ENABLE_BUF: U1.38, U5.2
- new net N$20: LED1.A, R6.1
- new net N$24: LED2.A, R7.1
- new net N$25: LED4.A, R9.1
- new net N$26: LED3.A, R8.1
- new net STAT_LED4: R6.2, U1.37
- new net STAT_LED5: R7.2, U1.36
- new net STAT_LED6: R8.2, U1.35
- new net STAT_LED7: R9.2, U1.34
- new net XTAL3: C11.2, Q2.1, R13.1, U3.5
- new net XTAL4: C12.2, Q2.2, R13.2, U3.4
- new net X_DIR: J10.8, U6.7
- new net X_MIN: R19.2, R26.1, U1.40
- new net X_STEP: J10.7, U6.6
- new net Y_DIR: J12.8, U7.7
- new net Y_MIN: R20.2, R25.1, U1.43
- new net Y_STEP: J12.7, U7.6
- new net Z_DIR: J14.8, U8.7
- new net Z_MIN: R21.2, R24.1, U1.44
- new net Z_STEP: J14.7, U8.6
- net !RESET!: now also J10.5; no longer J16.5
- net !SLEEP!: now also J10.6; no longer J16.6
- net +24V: now also J8.1, R43.2, TP3.1, U6.16, U6.30, U6.31, VR3.1, VR4.1, VR5.1; no longer Q2.1, Q3.1, Q4.1, R44.2, U9.16, U9.30, U9.31
- net +3V3: now also C2.1, J1.3, J2.1, J4.4, R17.2, R27.2, R28.2, R35.1, R38.2, R4.2, R41.2, R5.2, TP1.1, VR1.5; no longer J10.3, J12.4, J14.1, R19.2, R23.2, R24.2, R38.1, R39.2, R42.2
- net +5V: now also J5.2, J6.2, R42.2, TP2.1, VR2.4; no longer C1.1, C2.1, IC1.20, IC2.20, J1.2, J17.2, J2.2, J3.2, J7A.2, J8.2, J8A.2, J9.2, J9A.2, R2.2, R3.2, R4.1, R43.2, R5.1, R8.2, R9.2, TP4.1, U6.4
- net 1A_1: now also J11.5, U6.32; no longer J15.5, U7.32
- net 1A_2: now also J13.5, U7.32; no longer J18.5, U9.32
- net 1A_3: now also J15.5; no longer J4.5
- net 1B_1: now also J11.6, U6.34; no longer J15.6, U7.34
- net 1B_2: now also J13.6, U7.34; no longer J18.6, U9.34
- net 1B_3: now also J15.6; no longer J4.6
- net 2A_1: now also J11.4, U6.13; no longer J15.4, U7.13
- net 2A_2: now also J13.4, U7.13; no longer J18.4, U9.13
- net 2A_3: now also J15.4; no longer J4.4
- net 2B_1: now also J11.3, U6.15; no longer J15.3, U7.15
- net 2B_2: now also J13.3, U7.15; no longer J18.3, U9.15
- net 2B_3: now also J15.3; no longer J4.3
- net A: now also R39.2, R40.1; no longer R40.2, R41.1
- net B: now also R38.1, R40.2; no longer R39.1, R41.2
- net BRA: now also R44.2, U6.33; no longer R45.2, U7.33
- net BRA2: now also R46.2, U7.33; no longer R7.2, U9.33
- net BRB: now also R45.2, U6.14; no longer R46.2, U7.14
- net BRB2: now also U7.14; no longer U9.14
- net BRB3: now also R2.2; no longer R6.2
- net CLK: now also U6.1; no longer U9.1
- net CPI: now also U6.28; no longer U7.28
- net CPI2: now also U7.28; no longer U9.28
- net CPO: now also U6.27; no longer U7.27
- net CPO2: now also U7.27; no longer U9.27
- net DFU: now also R5.1, S3.2; no longer R24.1, S4.2
- net DTR: now also J1.6; no longer J10.6
- net ESTOP: now also U1.39
- net ESTOP_OE: now also J9.2, R27.1; no longer IC1.1, J31.2, R29.1
- net ETH_RX_ER: now also R17.1; no longer R18.1
- net GND: now also C1.1, C27.1, C75.1, J11.2, J11.8, J13.2, J13.8, J2.5, J2.9, J3.4, J4.6, J4.CD2, J4.GND1, J5.3, J6.3, LED1.C, LED2.C, LED3.C, LED4.C, LED5.C, LED6.C, LED7.C, R19.1, R2.1, R23.1, R29.1, R33.2, R39.1, R44.1, RJ2.SHLD0, RJ2.SHLD1, S1.1, TP4.1, U6.12, U6.18, U6.24, U6.35, U6.36, U6.PAD, VR2.3, VR2.5, VR2.GND, VR3.2, VR4.2, VR5.2; no longer C1.2, IC1.10, IC1.19, IC1.8, IC2.10, J1.3, J10.1, J10.2, J11.SHLD0, J11.SHLD1, J12.6, J12.CD2, J12.GND1, J13.4, J14.3, J14.5, J14.9, J17.3, J18.2, J18.8, J3.3, J4.2, J4.8, J7A.3, J8.3, J8A.3, J9.3, J9A.3, LED10.C, LED8.C, LED9.C, Q2.2, Q3.2, Q4.2, R17.1, R28.1, R33.1, R35.2, R40.1, R6.1, R7.1, S4.1, TP3.1, U6.3, U6.5, U6.GND, U9.12, U9.18, U9.24, U9.35, U9.36, U9.PAD
- net ISP_COM: now also R4.1, S2.2; no longer R23.1, S3.2
- net LED1/REGOFF: now also RJ2.9; no longer J11.9
- net LED2/NINTSEL: now also R23.2, RJ2.12; no longer J11.12, R33.2
- net MISO: now also J4.7, R36.2, U6.5; no longer J12.7, R37.2, U9.5
- net MOSI: now also J4.3, R35.2, U6.4; no longer J12.3, R36.2, U9.4
- net MS1: now also J10.2; no longer J16.2
- net MS2: now also J10.3; no longer J16.3
- net MS3: now also J10.4; no longer J16.4
- net N$10: now also LED7.A, R42.1; no longer LED9.A, R43.1
- net N$12: now also LED6.A, R43.1; no longer LED10.A, R44.1
- net N$14: now also VR2.2; no longer U6.2
- net N$17: now also VR1.2; no longer U5.2
- net N$5: now also J9.1, R29.2; no longer J31.1, R28.2
- net N$6: now also RJ2.4, RJ2.5; no longer J11.4, J11.5
- net N$7: now also R33.1, RJ2.11; no longer J11.11, R34.1
- net N$8: now also R34.1, RJ2.10; no longer J11.10, R35.1
- net N$9: now also LED5.A, R41.1; no longer LED8.A, R42.1
- net RD+: now also RJ2.3; no longer J11.3
- net RD-: now also RJ2.6; no longer J11.6
- net RESET: now also R18.1, S1.2; no longer R19.1, S2.2
- net RESET_N: now also J2.10; no longer J14.10
- net RTCK: now also J2.7; no longer J14.7
- net SCK: now also J4.5, U6.3; no longer J12.5, U9.3
- net SD_CS: now also J4.2, R37.2; no longer J12.2, R38.2
- net SPI_!CS1: now also U6.2; no longer U7.2
- net SPI_!CS2: now also U7.2; no longer U9.2
- net SWDCLK: now also J2.4; no longer J14.4
- net SWDIO: now also J2.2; no longer J14.2
- net SWO: now also J2.6; no longer J14.6
- net TD+: now also RJ2.1; no longer J11.1
- net TD-: now also RJ2.2; no longer J11.2
- net TDI: now also J2.8; no longer J14.8
- net USB_D+: now also J3.3; no longer J13.3
- net USB_D-: now also J3.2; no longer J13.2
- net VCC1: now also U6.26, U6.8, VR3.3; no longer Q2.3, U7.26, U7.8
- net VCC2: now also U7.26, U7.8, VR4.3; no longer Q4.3, U9.26, U9.8
- net VCC3: now also VR5.3; no longer Q3.3
- net VCP: now also U6.29; no longer U7.29
- net VCP2: now also U7.29; no longer U9.29
- net VR_IN: now also J3.1, VR1.1, VR1.3; no longer J13.1, U5.1, U5.3
- net VSW_IN: now also J8.2, VR2.1; no longer U6.1
- net XTAL1: now also C1.2, R3.1; no longer C11.2, R13.1, U3.5
- net XTAL2: now also C75.2, R3.2; no longer C12.2, R13.2, U3.4
- net X_STOP: now also J5.1, R26.2; no longer J7.1, J7A.1, R25.2
- net Y_STOP: now also J6.1, R25.2; no longer J8.1, J8A.1, R26.2
- net Z_STOP: now also J7.1, R24.2; no longer J9.1, J9A.1, R27.2
Routing:
- net +5V: track 371.8 -> 146.6 mm, vias 8 -> 1
- net Z_STOP: track 109.3 -> 2.35 mm, vias 2 -> 0
- net !X_ENABLE: track 93.1 -> 0.00 mm, vias 4 -> 0
- net X_STOP: track 95.6 -> 5.40 mm, vias 2 -> 0
- net AVR_TXD: track 61.6 -> 0.00 mm, vias 4 -> 0
- net AVR_RXD: track 59.6 -> 0.00 mm, vias 2 -> 0
- net !Z_ENABLE: track 56.1 -> 0.00 mm, vias 2 -> 0
- net IOREF: track 53.1 -> 0.00 mm
- net !Z_ENABLE_BUF: track 52.8 -> 0.00 mm, vias 4 -> 0
- net !Y_ENABLE: track 43.6 -> 0.00 mm, vias 3 -> 0
- net !ENABLE: track 0.00 -> 41.8 mm, vias 0 -> 3
- net !X_ENABLE_BUF: track 37.8 -> 0.00 mm, vias 1 -> 0
- net SERVO1: track 36.5 -> 0.00 mm
- net SERVO2: track 33.8 -> 0.00 mm
- net SERVO4: track 33.7 -> 0.00 mm
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