File: EAGLE/EMC03 - Motion Control/EMC03-Motion Control.brd (EAGLE design)
At the start: 100 x 86.6 mm, 209 parts, among them J1 UART0, J10 S4B-PH-SM4, J11 S4B-PH-SM4, J12 S4B-PH-SM4, J13 S5B-PH-SM4, J14 S5B-PH-SM4, J15 S5B-PH-SM4, J16 S8B-PH-SM4, J17 S8B-PH-SM4, J18 S6B-PH-SM4, J19 S6B-PH-SM4, J2 FTSH-105-1-L-DV, J3 USB-B, J4 MicroSD, J5 S3B-PH-SM4, J6 S3B-PH-SM4, J7 S3B-PH-SM4, J8 694106106102, J9 S2B-PH-SM4, Q1 12MHz, Q2 25MHz, U1 LPC1768, U2 SP3485, U3 LAN8720A, U4 74LVC1G04W5-7, U5 74AHCT, U6 TMC2130-LA, U7 TMC2130-LA, U8 TMC2130-LA

Commit message: Arranged EMC03 board as much as possible. Updated PCB Checklist with testpoint data. Updated test points to pads, as per schematic instructions.
Parts:
- TP1, TP2, TP3, TP4: device FirePick:CON-TESTPOINT -> TinWhiskers:TESTPAD
- moved RJ1 398.8 mm to (63.2, 95.7)
- moved FB2 265.7 mm to (279.3, -192.9), turned to 180 degrees
- moved R5 261.8 mm to (279.3, -452.7), turned to 180 degrees
- moved C29 194.8 mm to (209.4, -194.1)
- moved LED4 194.8 mm to (209.4, -324.0)
- moved S2 194.8 mm to (209.4, -259.1)
- moved C25 149.5 mm to (587.8, 68.1)
- moved C32 149.5 mm to (587.8, 3.17)
- moved FB1 149.5 mm to (587.8, -61.8)
- moved Q2 149.5 mm to (587.8, 133.1)
- moved R12 149.5 mm to (587.8, 263.0)
- moved R31 149.5 mm to (587.8, 327.9)
- moved R36 149.5 mm to (587.8, 198.0)
- moved LED3 139.5 mm to (279.3, -257.8), turned to 180 degrees
- moved C28 135.8 mm to (279.3, -387.7), turned to 180 degrees
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Connections:
- net +24V: now also TP3.PAD; no longer TP3.1
- net +3V3: now also TP1.PAD; no longer TP1.1
- net +5V: now also TP2.PAD; no longer TP2.1
- net GND: now also TP4.PAD; no longer TP4.1
Other:
- board text added: "ENCODER"

Commit message: Updated schematic to integrate Intel Edison into EMC03 (USB chip for serial console, USB hub for all peripherals and associated EEPROM, second RS-485 transceiver for Edison). USB-B connection has been removed and replaced with a panel-mount version connected by vertical header. Ethernet interface connects to USB hub now, and MicroSD interfaces with Edison instead of LPC1768. Some of the 5V switching regulators have been removed for the time being. All necessary parts for EMC03 have been added to TinWhiskers library. EFD01 Schematic has a complete set of connections, could use some tidying up before layout.
Parts:
- removed C60, C73: 0.33uF, TinWhiskers:C0603
- removed C61, C74: 100 nF, TinWhiskers:C0603
- removed R35, R37: 10K, TinWhiskers:R0603
- removed R36: 10k, TinWhiskers:R0603
- removed VR3, VR4, VR5: KA78L05AMTF, TinWhiskers:SOT-89
- added C77, C79, C80, C81, C82, C84, C85, C87: 0.1uF, TinWhiskers:C0603
- added C78: 10nF, TinWhiskers:C0603
- added C83: 4.7uF, TinWhiskers:C0603
- added C86: 1.0uF, TinWhiskers:C0603
- added D15: SJPB-H6, TinWhiskers:DIO-SM2
- added FB3, FB4: 120R, TinWhiskers:F0603
- added J20: Intel EDISON, TinWhiskers:DF40HC(3.0)-70DS-0.4V(51)
- added J21: PWRBUTTON, TinWhiskers:CON-HDR-2POS-MALE
- added J22: SERIAL CONS., TinWhiskers:CON-HDR-4POS-MALE
- added J23: LCD, TinWhiskers:CON-HDR-4POS-MALE
- added L2: 100uH, TinWhiskers:L-SMD-12.5MM
- added LED11, LED8, LED9: GREEN, TinWhiskers:LED0603
- added R48: 10K, TinWhiskers:R0603
- added R49, R50: 1K, TinWhiskers:R0603
- added R51: 120R, TinWhiskers:R0603
- added R52: 1.5K, TinWhiskers:R0603
- added R53, R54: 270R, TinWhiskers:R0603
- added U10: FT232RL, TinWhiskers:28-SSOP
- added U11, U12, U13, U14, U15: 74LVC1T45, TinWhiskers:SOT-363
- added U16: TXS0206-29, TinWhiskers:20-XFBGA
- added U9: SP3485, TinWhiskers:SOICN-8
- C11, C12: value 12pF -> 33pF
- C14, C22: value 10uF -> 0.1uF; device TinWhiskers:C-RAD-6.3MM -> TinWhiskers:C0603
- C20: value 1uF -> 0.1uF; device TinWhiskers:C-SMD-4MM -> TinWhiskers:C0603
- C21: value 470pF -> 0.1uF
- C33, C35: value 1uF -> 0.1uF
- C36: value 1uF -> 220uF; device TinWhiskers:C0603 -> TinWhiskers:C-SMD-10MM
- C50: value 0.33uF -> 470uF; device TinWhiskers:C0603 -> TinWhiskers:C-SMD-10MM
- C51: value 100 nF -> 0.47uF
- FB1, FB2: value BLM18AG121SN1D -> 120R
- J3: value USB-B -> USB-A; device TinWhiskers:USB-B(THRU) -> TinWhiskers:CON-HDR-4POS-MALE
- J4: value MicroSD -> USD-SOCKET
- R10: value 22R -> 330R
- R11: value 22R -> 1M
- R12: value 22R -> 825R
- R13: value 1M -> 12.4K
- R14: value 12.1K -> 10K
- R15: value 22R -> 0R1
- R16: value 1.5K -> DNP
- R17, R23: value 10K -> 10.5K
- R40: value 100R -> 120R
- U3: value LAN8720A -> 93LC66A; device TinWhiskers:QFN-24 -> TinWhiskers:SOT-23-6
- U4: value 74LVC1G04W5-7 -> LAN9514; device TinWhiskers:SOT-25 -> TinWhiskers:64-QFN
- VR1: value TC1015-3.3VCT713 -> SI-8033JD; device TinWhiskers:SOT-23-5 -> TinWhiskers:TO263-5
- moved R17 1714.9 mm to (-747.9, -769.5)
- moved C22 1702.2 mm to (-718.0, -688.9)
- moved R14 1683.8 mm to (-718.4, -627.7)
- moved C14 1670.6 mm to (-718.0, -663.9)
- moved R16 1664.9 mm to (-718.4, -754.0)
- moved R15 1645.8 mm to (-718.4, -750.5)
- moved R13 1594.4 mm to (-718.4, -624.2)
- moved R12 1577.0 mm to (-718.4, -620.7)
- moved C19 1572.2 mm to (-718.0, -673.9)
- moved C36 1566.0 mm to (-729.7, -806.7)
- moved C33 1562.4 mm to (-747.5, -776.6)
- moved C21 1556.1 mm to (-718.0, -683.9)
- moved C18 1552.0 mm to (-718.0, -668.9)
- moved C35 1551.2 mm to (-747.5, -781.6)
- moved C13 1528.6 mm to (-718.0, -658.9)
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Connections:
- net DI renamed DI1
- net RO renamed RO1
- removed net CRSPIN: R12.2, U3.11
- removed net ETH_CRS_DV: R12.1, U1.92
- removed net ETH_MDC: U1.87, U3.13
- removed net ETH_MDIO: R16.1, U1.86, U3.12
- removed net ETH_REF_CLK: R15.1, U1.88
- removed net ETH_RXD0: R10.1, U1.91
- removed net ETH_RXD1: R11.1, U1.90
- removed net ETH_RX_ER: R17.1, U1.89, U3.10
- removed net ETH_TXD0: U1.95, U3.17
- removed net ETH_TXD1: U1.94, U3.18
- removed net ETH_TX_EN: U1.93, U3.16
- removed net LED1/REGOFF: RJ1.9, U3.3
- removed net LED2/NINTSEL: R23.2, RJ1.12, U3.2
- removed net N$23: C20.POS, C21.2, U3.6
- removed net NINT/REFCLK0: U3.14, U4.2
- removed net NRST: U3.15
- removed net RBIAS: R14.2, U3.24
- removed net RXD0PIN: R10.2, U3.8
- removed net RXD1PIN: R11.2, U3.7
- removed net SD_CS: J4.2, R37.2, U1.79
- removed net USB_D+: J3.3, U1.29
- removed net USB_D-: J3.2, U1.30
- removed net VCC1: C51.2, U6.26, U6.8, VR3.3
- removed net VCC2: C74.2, U7.26, U7.8, VR4.3
- removed net VCC3: C61.2, U8.26, U8.8, VR5.3
- removed net VR_IN: J3.1, VR1.1, VR1.3
- removed net XTAL3: C11.2, Q2.1, R13.1, U3.5
- removed net XTAL4: C12.2, Q2.2, R13.2, U3.4
- new net !PWRBTN: J20.17, J21.1, R48.1
- new net !RXLED: LED9.C, U10.22
- new net !TXLED: LED8.C, U10.23
- new net +1V8: C35.2, J20.12, R17.2, R23.2, U11.6, U12.1, U13.1, U14.1, U15.6, U16.A2
- new net CLKA: J20.58, U16.D2
- new net CLKB: J4.5, U16.D3
- new net CLKF: J20.44, U16.E2
- new net CMD: J4.3
- new net CMDA: J20.62, U16.C1
- new net CMDB: U16.C4
- new net DAT0A: J20.66, U16.D1
- new net DAT0B: J4.7, U16.D4
- new net DAT1A: J20.70, U16.E1
- new net DAT1B: J4.8, U16.E4
- new net DAT2: J4.1
- new net DAT2A: J20.64, U16.A1
- new net DAT2B: U16.A4
- new net DAT3: J4.2
- new net DAT3A: J20.68, U16.B1
- new net DAT3B: U16.B4
- new net DI2: J20.46, U13.3
- new net DI2O: U13.4, U9.4
- new net DM: J22.3, U10.16
- new net DP: J22.2, R52.1, U10.15
- new net EECLK: U3.4, U4.23
- new net EECS: U3.5, U4.24
- new net EEDI: U3.1, U4.26
- new net EEDO: U3.3, U4.25
- new net EN: R17.1, U16.E3
- new net LED_DUPLEX: LED11.C, U4.20
- new net LED_SPEED: RJ1.12, U4.22
- new net LED_TXRX: RJ1.9, U4.21
- new net N$1: C77.2, U10.17
- new net N$11: LED9.A, R54.1
- new net N$13: LED8.A, R53.1
- new net N$15: R13.2, U4.50
- new net N$16: D15.POS, L2.P$1, VR1.2
- new net N$18: R14.1, U4.41
- new net N$2: C78.2, FB3.1, J22.1
- new net N$21: J20.14, J20.2, J20.4, J20.6, R15.1, R16.1
- new net RO2: U15.3, U9.1
- new net RO2O: J20.61, U15.4
- new net RTS: J20.63, U14.3
- new net RTSO: U14.4, U9.2, U9.3
- new net RXD: U10.5, U11.3
- new net RXDO: J20.22, U11.4
- new net SD_CD: J20.60, J4.CD1, R23.1, U16.A3
- new net TXD: J20.27, U12.3
- new net TXDO: U10.1, U12.4
- new net USBA_D+: J3.3, U4.7
- new net USBA_D-: J3.2, U4.6
- new net USBDM0: J20.18, U4.58
- new net USBDP0: J20.16, U4.59
- new net USBMCU+: U1.29, U4.9
- new net USBMCU-: U1.30, U4.8
- new net VCCB: C34.2, J4.4, U16.B3
- new net VDD18C: C83.2, C84.2, C85.2, U4.15, U4.38
- new net VDD18ETH: C87.2, FB4.2, U4.48
- new net VDD18USB: C86.2, FB4.1, U4.62
- new net VDD33A: C13.2, C14.2, C18.2, C19.2, C20.2, C21.2, C22.2, FB1.1, U4.10, U4.49, U4.5, U4.51, U4.54, U4.57, U4.64
- new net XI: C12.2, Q2.2, R11.2, U4.61
- new net XO: C11.2, Q2.1, R11.1, U4.60
- net +24V: no longer C50.2, C60.2, C73.2, VR3.1, VR4.1, VR5.1
- net +3V3: now also C24.2, C25.2, C50.POS, C79.2, C80.2, C81.2, C82.2, FB1.2, FB3.2, L2.P$2, R10.2, R12.2, R14.2, R15.2, R22.2, R30.2, R31.2, R32.2, R48.2, R49.2, R52.2, R53.2, R54.2, RJ1.4, RJ1.5, U10.19, U10.20, U10.4, U11.1, U12.6, U13.6, U14.6, U15.1, U16.B2, U3.6, U4.19, U4.27, U4.33, U4.39, U4.40, U4.46, U9.8, VR1.4; no longer C13.2, C22.POS, C34.2, C36.2, FB1.1, J4.4, R17.2, R35.1, R36.1, R37.1, U3.9, U4.5, VR1.5
- net +5V: now also C36.POS, J3.1, U6.26, U6.8, U7.26, U7.8, U8.26, U8.8, VR1.1
- net A: now also R50.2, R51.1, U9.6
- net B: now also R49.1, R51.2, U9.7
- net EE_D+: now also U4.2
- net EE_D-: now also U4.1
- net GND: now also C14.1, C20.1, C22.1, C36.NEG, C50.NEG, C77.1, C78.1, C79.1, C80.1, C81.1, C82.1, C83.1, C84.1, C85.1, C86.1, C87.1, D15.NEG, J20.1, J20.11, J20.13, J20.15, J20.5, J20.9, J21.2, J22.4, J4.GND2, R13.1, R50.1, U10.18, U10.21, U10.25, U10.26, U10.7, U11.2, U11.5, U12.2, U12.5, U13.2, U13.5, U14.2, U14.5, U15.2, U15.5, U16.C2, U16.C3, U3.2, U4.34, U4.44, U4.PAD, U9.5, VR1.3, VR1.GND; no longer C14.NEG, C20.NEG, C22.NEG, C36.1, C50.1, C60.1, C61.1, C73.1, C74.1, R14.1, R23.1, U3.PAD, U4.3, VR3.2, VR4.2, VR5.2
- net ISP_COM: now also U1.53; no longer U1.48
- net MISO: no longer J4.7, R36.2
- net MOSI: no longer J4.3, R35.2
- net N$17: now also C51.2, VR1.5; no longer C35.2, VR1.2
- net N$3: now also LED11.A, R10.1; no longer R15.2, U4.4
- net N$6: now also R12.1, U4.11; no longer C14.POS, C18.2, C19.2, C24.2, C25.2, FB1.2, R22.2, R30.2, R31.2, R32.2, RJ1.4, RJ1.5, U3.1, U3.19
- net RD+: now also U4.52; no longer U3.23
- net RD-: now also U4.53; no longer U3.22
- net RESET: now also U4.12
- net SCK: no longer J4.5
- net TD+: now also U4.55; no longer U3.21
- net TD-: now also U4.56; no longer U3.20
- net ULC_D+: now also U4.4
- net ULC_D-: now also U4.3

Commit message: Updated schematic to incorporate tweaks proposed by Neil. Generated new and complete BOM, updated parts database.
Parts:
- removed C86: 1.0uF, TinWhiskers:C0603
- removed C87: 0.1uF, TinWhiskers:C0603
- added C60, C74: 0.1uF, TinWhiskers:C0603
- added C61: 4.7uF, TinWhiskers:C0603
- added C73: 1.0uF, TinWhiskers:C0603
- added LED10, LED12, LED13, LED14: GREEN, TinWhiskers:LED0603
- added R35: 12K, TinWhiskers:R0603
- added R36: 0R, TinWhiskers:R0603
- added R37, R55, R56: 511R, TinWhiskers:R0603
- added R57: 0R1, TinWhiskers:R0603
- added R58: DNP, TinWhiskers:R0603
- added U18, U19: MIC2026-1YM, TinWhiskers:SOIC-8
- J4: value USD-SOCKET -> 47334-0001
- J9: value S2B-PH-SM4 -> ESTOP
- R52: value 1.5K -> 511R
- U10: value FT232RL -> FT231XS-R; device TinWhiskers:28-SSOP -> TinWhiskers:20-SSOP
- VR1: value SI-8033JD -> SI-8050JD
- VR2: value SI-8050JD -> SI-8033JD
- moved J4 1153.0 mm to (57.1, 96.9)
- moved VR1 1027.6 mm to (-65.0, -65.0)
- moved C33 743.0 mm to (-468.0, -88.2)
- moved C35 743.0 mm to (-468.0, -93.2)
- moved C77 743.0 mm to (-435.5, 179.4)
- moved FB3 743.0 mm to (-438.7, 174.9)
- moved FB4 743.0 mm to (-439.1, -58.4)
- moved J20 743.0 mm to (-429.2, 225.9)
- moved J21 743.0 mm to (-434.7, 222.0)
- moved L2 743.0 mm to (-462.9, -121.8)
- moved R14 743.0 mm to (-438.9, 60.7)
- moved R17 743.0 mm to (-468.4, -81.0)
- moved R23 743.0 mm to (-468.4, -84.5)
- moved R53 743.0 mm to (-438.5, 166.2)
- moved R54 743.0 mm to (-438.5, 162.7)
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Connections:
- net N$15 renamed EXRES
- new net !DTR: U10.1
- new net !RESET: R36.1
- new net N$15: R36.2, U4.12
- new net N$19: J20.12, R57.2, R58.2
- new net N$27: R35.2, U4.63
- new net N$28: LED10.A, R37.1
- new net N$29: LED12.A, R52.1
- new net N$30: LED13.A, R55.1
- new net N$31: LED14.A, R56.1
- new net PRTCTL2: U18.1, U18.2, U4.14
- new net PRTCTL3: U18.3, U18.4, U4.16
- new net PRTCTL4: U19.1, U19.2, U4.17
- new net PRTCTL5: U19.3, U19.4, U4.18
- new net PWR1: J16.6, R56.2, U18.8
- new net PWR2: J17.6, R55.2, U18.5
- new net PWR3: J3.1, R52.2, U19.8
- new net PWR4: R37.2, U19.5
- net !RXLED: no longer U10.22
- net !TXLED: no longer U10.23
- net +1V8: now also R57.1, R58.1; no longer J20.12
- net +24V: now also VR1.1; no longer VR2.1
- net +3V3: now also C60.2, C61.2, VR2.4; no longer R52.2, U10.19, U10.20, U10.4, VR1.4
- net +5V: now also U18.7, U19.7, VR1.4, VR2.1; no longer J16.6, J17.6, J3.1, VR1.1, VR2.4
- net CLK: now also U1.33
- net DM: no longer U10.16
- net DP: no longer R52.1, U10.15
- net EE_D+: now also U4.4; no longer U4.2
- net EE_D-: now also U4.3; no longer U4.1
- net GND: now also C60.1, C61.1, C73.1, C74.1, LED10.C, LED12.C, LED13.C, LED14.C, R35.1, U18.6, U19.6; no longer C86.1, C87.1, U10.18, U10.21, U10.25, U10.26, U10.7
- net N$1: no longer U10.17
- net N$14: now also VR1.2; no longer VR2.2
- net N$16: now also VR2.2; no longer VR1.2
- net N$17: now also VR2.5; no longer VR1.5
- net N$4: now also VR1.5; no longer VR2.5
- net RESET: no longer U4.12
- net RXD: no longer U10.5
- net TXDO: no longer U10.1
- net ULC_D+: now also U4.2; no longer U4.4
- net ULC_D-: now also U4.1; no longer U4.3
- net VDD18ETH: now also C74.2; no longer C87.2
- net VDD18USB: now also C73.2; no longer C86.2

Commit message: Preliminary final draft for EMC03, ECAM02, and EFD01 boards.
Parts:
- added U17, U20: 74LVC, TinWhiskers:SOT-23-5
- added U21, U22: 74LVC1T45, TinWhiskers:SOT-363
- J23: value LCD -> B14B-PH; device TinWhiskers:CON-HDR-4POS-MALE -> TinWhiskers:CONN-JST-PH-2.0MM-14P-VRT
- J4: value 47334-0001 -> 101-00581-59; device TinWhiskers:MICRO-SD-SOCKET-PP -> TinWhiskers:MICRO-SD-SOCKET-AMPH
- moved J4 992.4 mm to (-723.1, -516.5)
Connections:
- new net EEEN: U22.3
- new net EEENO: U17.1, U22.4
- new net LCD_CS: J20.39, J23.11
- new net LCD_D0: J20.52, J23.3
- new net LCD_D1: J20.54, J23.4
- new net LCD_D2: J20.50, J23.5
- new net LCD_D3: J20.56, J23.6
- new net LCD_D4: J20.24, J23.7
- new net LCD_D5: J20.26, J23.8
- new net LCD_D6: J20.28, J23.9
- new net LCD_D7: J20.30, J23.10
- new net LCD_RD: J20.37, J23.14
- new net LCD_RS: J20.34, J23.12
- new net LCD_WR: J20.32, J23.13
- new net N$22: U17.4, U18.1
- new net N$42: U18.4, U20.4
- new net ULCEN: U21.3
- new net ULCENO: U20.1, U21.4
- net +1V8: now also U21.1, U22.1
- net +3V3: now also J23.1, U17.5, U20.5, U21.6, U22.6
- net GND: now also J23.2, J4.GND, J4.NC, U17.3, U20.3, U21.2, U21.5, U22.2, U22.5; no longer J4.CD2, J4.GND1
- net PRTCTL2: now also U17.2; no longer U18.1
- net PRTCTL3: now also U20.2; no longer U18.4
- net SD_CD: now also J4.CD; no longer J4.CD1

Commit message: Component placement begun
Parts:
- moved LED10 980.6 mm to (132.8, 9.29)
- moved LED12 980.6 mm to (132.8, 4.54)
- moved LED13 980.6 mm to (132.8, -0.21)
- moved LED14 980.6 mm to (132.8, -4.96)
- moved R36 980.6 mm to (131.3, -26.7)
- moved R37 980.6 mm to (131.3, 23.2)
- moved R52 980.6 mm to (131.3, 19.7)
- moved R55 980.6 mm to (131.3, 16.1)
- moved R56 980.6 mm to (131.3, 12.6)
- moved R57 980.6 mm to (131.3, -9.87)
- moved R58 980.6 mm to (131.3, -13.4)
- moved U18 980.6 mm to (133.5, 34.9)
- moved U19 980.6 mm to (133.5, 28.5)
- moved U17 980.0 mm to (117.8, -32.6)
- moved U20 980.0 mm to (117.8, -36.9)
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Routing:
- net RESET: track 0.00 -> 11.7 mm
- net DTR: track 0.00 -> 4.57 mm
Other:
- board text removed: "3.3V I/O"
- board text removed: "5V I/O"

Commit message: Preliminary placement and routing done for EFD01. Preliminary placement done for EMC03. All schematics are ready for review (A0 for ECAM03 needs to be defined, also SS for EFD01, ECAM03, etc.)
Parts:
- moved U15 222.7 mm to (61.2, 65.1), flipped to the bottom, turned to 315 degrees
- moved U14 219.4 mm to (58.9, 67.5), flipped to the bottom, turned to 135 degrees
- moved U11 218.2 mm to (63.3, 57.6), flipped to the bottom, turned to 315 degrees
- moved U12 217.1 mm to (63.8, 62.7), flipped to the bottom, turned to 315 degrees
- moved U13 215.7 mm to (58.2, 62.3), flipped to the bottom, turned to 315 degrees
- moved C19 206.8 mm to (36.8, 65.2), turned to 225 degrees
- moved C18 204.4 mm to (35.7, 66.7), turned to 225 degrees
- moved C14 202.8 mm to (39.5, 58.4), turned to 135 degrees
- moved C13 202.7 mm to (40.9, 59.7), turned to 135 degrees
- moved R12 197.5 mm to (44.7, 59.3), flipped to the bottom, turned to 270 degrees
- moved C61 193.7 mm to (70.4, 34.8)
- moved R13 191.6 mm to (36.9, 65.4), flipped to the bottom, turned to 315 degrees
- moved C60 189.4 mm to (67.3, 35.6)
- moved FB4 188.6 mm to (38.7, 67.5), flipped to the bottom, turned to 45 degrees
- moved R14 184.8 mm to (28.8, 66.8), flipped to the bottom, turned to 135 degrees
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Connections:
- net EEEN: now also J20.48
- net ULCEN: now also J20.42
Routing:
- net RESET: track 11.7 -> 0.00 mm
- net DTR: track 4.57 -> 0.00 mm
Other:
- board text added: "USB-A"

Commit message: Split the EMC03 into EMC03 and EFP01 (front panel board) to make routing 10000000x easier
Parts:
- removed C13, C14, C18, C19, C20, C21, C22, C23, C24, C25, C33, C34, C35, C4, C60, C74, C77, C79, C80, C81, C82, C84, C85: 0.1uF, TinWhiskers:C0603
- removed C26, C30, C31, C32: 18pF, TinWhiskers:C0603
- removed C3: 100uF, rcl:PANASONIC_D
- removed C37: 220uF, TinWhiskers:C-SMD-10MM
- removed C38: 470uF, TinWhiskers:C-SMD-10MM
- removed C61, C83: 4.7uF, TinWhiskers:C0603
- removed C73: 1.0uF, TinWhiskers:C0603
- removed C76: 0.47uF, TinWhiskers:C0603
- removed C78: 10nF, TinWhiskers:C0603
- removed D2: SJPB-H6, TinWhiskers:DIO-SM2
- removed FB1, FB3, FB4: 120R, TinWhiskers:F0603
- removed FID1, FID2, FID3, FID4, FID5, FID6, FID7: FIDUCIAL, FirePick:FIDUCIAL
- removed J20: Intel EDISON, TinWhiskers:DF40HC(3.0)-70DS-0.4V(51)
- removed J21: PWRBUTTON, TinWhiskers:CON-HDR-2POS-MALE
- removed J22: SERIAL CONS., TinWhiskers:CON-HDR-4POS-MALE
- removed J23: B14B-PH, TinWhiskers:CONN-JST-PH-2.0MM-14P-VRT
- removed J8: 694106106102, TinWhiskers:PJ-694106106102
- removed L1: 100uH, TinWhiskers:L-SMD-12.5MM
- removed LED10, LED11, LED12, LED13, LED14, LED8, LED9: GREEN, TinWhiskers:LED0603
- removed LED6, LED7: RED, TinWhiskers:LED0603
- removed LOGO4: LOGO-FIREPICKLARGE, FirePick:LOGO-FIREPICK
- removed LOGO5: LOGO-OSHWMEDIUM, FirePick:LOGO-OSHW-MEDIUM
- removed LOGO6: LOGO-CC-BY-SALARGE, FirePick:LOGO-CC-BY-SA
- removed Q2: 25MHz, TinWhiskers:HC-49/U-S
- removed R11: 1M, TinWhiskers:R0603
- removed R12: 825R, TinWhiskers:R0603
- removed R13: 12.4K, TinWhiskers:R0603
- removed R14, R43, R48: 10K, TinWhiskers:R0603
- removed R15, R57: 0R1, TinWhiskers:R0603
- removed R16, R58: DNP, TinWhiskers:R0603
- removed R17, R23: 10.5K, TinWhiskers:R0603
- removed R22, R30, R31, R32: 49R9, TinWhiskers:R0603
- removed R33, R34: 330R, TinWhiskers:R0603
- removed R35: 12K, TinWhiskers:R0603
- removed R36: 0R, TinWhiskers:R0603
- removed R37, R52, R55, R56: 511R, TinWhiskers:R0603
- removed R42: 1.2K, TinWhiskers:R0603
- removed R49, R50: 1K, TinWhiskers:R0603
- removed R51: 120R, TinWhiskers:R0603
- removed R53, R54: 270R, TinWhiskers:R0603
- removed RJ1: HR911105A, TinWhiskers:MAGJACK(HR911105A)
- removed TP2: +5V, TinWhiskers:TESTPAD
- removed U$25: TIN-WHISKERSTSTOP, !tin-whiskers:TIN-WHISKERS-TSTOP
- removed U10: FT231XS-R, TinWhiskers:20-SSOP
- removed U11, U12, U13, U14, U15, U21, U22: 74LVC1T45, TinWhiskers:SOT-363
- removed U16: TXS0206-29, TinWhiskers:20-XFBGA
- removed U17, U20: 74LVC, TinWhiskers:SOT-23-5
- removed U18, U19: MIC2026-1YM, TinWhiskers:SOIC-8
- removed U3: 93LC66A, TinWhiskers:SOT-23-6
- removed U4: LAN9514, TinWhiskers:64-QFN
- removed U9: SP3485, TinWhiskers:SOICN-8
- removed VR1: SI-8050JD, TinWhiskers:TO263-5
- C11: value 33pF -> 4.7 uF
- C12: value 33pF -> 4.7uF
- J3: value USB-A -> CONN-OSTTH050160; device TinWhiskers:CON-HDR-4POS-MALE -> FirePick:CONN-OSTTH050160
- J4: value 101-00581-59 -> (none); device TinWhiskers:MICRO-SD-SOCKET-AMPH -> !con-lstb:MA07-2
- R10: value 330R -> 2.2; device TinWhiskers:R0603 -> TinWhiskers:R1206
- moved C12 185.3 mm to (-94.0, -72.8), flipped to the top, turned to 0 degrees
- moved C50 178.6 mm to (61.2, 68.7)
- moved C11 175.5 mm to (-94.0, -67.7), flipped to the top, turned to 0 degrees
- moved C36 166.0 mm to (63.4, 81.3), turned to 90 degrees
- moved VR2 164.3 mm to (41.2, 66.5), turned to 90 degrees
- moved R10 157.9 mm to (-93.9, -63.9), turned to 0 degrees
- moved L2 157.2 mm to (40.1, 81.0)
- moved U8 98.5 mm to (23.8, 59.6)
- moved U7 80.0 mm to (51.3, 23.1)
- moved U6 64.7 mm to (72.5, 58.9)
- moved J2 50.4 mm to (65.6, 29.1)
- moved J3 42.2 mm to (50.7, 90.6), turned to 0 degrees
- moved J4 27.6 mm to (34.3, -3.05), flipped to the top, turned to 0 degrees
Connections:
- removed net !DTR: U10.1
- removed net !PWRBTN: J20.17, J21.1, R48.1
- removed net !RESET: R36.1
- removed net !RXLED: LED9.C
- removed net !TXLED: LED8.C
- removed net +1V8: C35.2, R17.2, R23.2, R57.1, R58.1, U11.6, U12.1, U13.1, U14.1, U15.6, U16.A2, U21.1, U22.1
- removed net CLKA: J20.58, U16.D2
- removed net CLKB: J4.5, U16.D3
- removed net CLKF: J20.44, U16.E2
- removed net CMD: J4.3
- removed net CMDA: J20.62, U16.C1
- removed net CMDB: U16.C4
- removed net DAT0A: J20.66, U16.D1
- removed net DAT0B: J4.7, U16.D4
- removed net DAT1A: J20.70, U16.E1
- removed net DAT1B: J4.8, U16.E4
- removed net DAT2: J4.1
- removed net DAT2A: J20.64, U16.A1
- removed net DAT2B: U16.A4
- removed net DAT3: J4.2
- removed net DAT3A: J20.68, U16.B1
- removed net DAT3B: U16.B4
- removed net DI2: J20.46, U13.3
- removed net DI2O: U13.4, U9.4
- removed net DM: J22.3
- removed net DP: J22.2
- removed net EECLK: U3.4, U4.23
- removed net EECS: U3.5, U4.24
- removed net EEDI: U3.1, U4.26
- removed net EEDO: U3.3, U4.25
- removed net EEEN: J20.48, U22.3
- removed net EEENO: U17.1, U22.4
- removed net EN: R17.1, U16.E3
- removed net EXRES: R13.2, U4.50
- removed net LCD_CS: J20.39, J23.11
- removed net LCD_D0: J20.52, J23.3
- removed net LCD_D1: J20.54, J23.4
- removed net LCD_D2: J20.50, J23.5
- removed net LCD_D3: J20.56, J23.6
- removed net LCD_D4: J20.24, J23.7
- removed net LCD_D5: J20.26, J23.8
- removed net LCD_D6: J20.28, J23.9
- removed net LCD_D7: J20.30, J23.10
- removed net LCD_RD: J20.37, J23.14
- removed net LCD_RS: J20.34, J23.12
- removed net LCD_WR: J20.32, J23.13
- removed net LED_DUPLEX: LED11.C, U4.20
- removed net LED_SPEED: RJ1.12, U4.22
- removed net LED_TXRX: RJ1.9, U4.21
- removed net N$10: LED7.A, R42.1
- removed net N$11: LED9.A, R54.1
- removed net N$12: LED6.A, R43.1
- removed net N$13: LED8.A, R53.1
- removed net N$14: D2.POS, L1.P$1, VR1.2
- removed net N$15: R36.2, U4.12
- removed net N$18: R14.1, U4.41
- removed net N$19: J20.12, R57.2, R58.2
- removed net N$21: J20.14, J20.2, J20.4, J20.6, R15.1, R16.1
- removed net N$22: U17.4, U18.1
- removed net N$27: R35.2, U4.63
- removed net N$28: LED10.A, R37.1
- removed net N$29: LED12.A, R52.1
- removed net N$3: LED11.A, R10.1
- removed net N$30: LED13.A, R55.1
- removed net N$31: LED14.A, R56.1
- removed net N$4: C76.2, VR1.5
- removed net N$42: U18.4, U20.4
- removed net N$6: R12.1, U4.11
- removed net N$7: R33.1, RJ1.11
- removed net N$8: R34.1, RJ1.10
- removed net PRTCTL2: U17.2, U18.2, U4.14
- removed net PRTCTL3: U18.3, U20.2, U4.16
- removed net PRTCTL4: U19.1, U19.2, U4.17
- removed net PRTCTL5: U19.3, U19.4, U4.18
- removed net PWR3: J3.1, R52.2, U19.8
- removed net PWR4: R37.2, U19.5
- removed net RD+: C31.2, R31.1, RJ1.3, U4.52
- removed net RD-: C32.2, R32.1, RJ1.6, U4.53
- removed net RO2: U15.3, U9.1
- removed net RO2O: J20.61, U15.4
- removed net RTS: J20.63, U14.3
- removed net RTSO: U14.4, U9.2, U9.3
- removed net RXD: U11.3
- removed net RXDO: J20.22, U11.4
- removed net SD_CD: J20.60, J4.CD, R23.1, U16.A3
- removed net TD+: C26.2, R22.1, RJ1.1, U4.55
- removed net TD-: C30.2, R30.1, RJ1.2, U4.56
- removed net TXD: J20.27, U12.3
- removed net TXDO: U12.4
- removed net ULCEN: J20.42, U21.3
- removed net ULCENO: U20.1, U21.4
- removed net USBA_D+: J3.3, U4.7
- removed net USBA_D-: J3.2, U4.6
- removed net USBDM0: J20.18, U4.58
- removed net USBDP0: J20.16, U4.59
- removed net VCCB: C34.2, J4.4, U16.B3
- removed net VDD18C: C83.2, C84.2, C85.2, U4.15, U4.38
- removed net VDD18ETH: C74.2, FB4.2, U4.48
- removed net VDD18USB: C73.2, FB4.1, U4.62
- removed net VDD33A: C13.2, C14.2, C18.2, C19.2, C20.2, C21.2, C22.2, FB1.1, U4.10, U4.49, U4.5, U4.51, U4.54, U4.57, U4.64
- removed net XI: C12.2, Q2.2, R11.2, U4.61
- removed net XO: C11.2, Q2.1, R11.1, U4.60
- net +24V: no longer C37.POS, J8.2, R43.2, VR1.1
- net +3V3: no longer C23.2, C24.2, C25.2, C33.2, C60.2, C61.2, C79.2, C80.2, C81.2, C82.2, FB1.2, FB3.2, J23.1, R10.2, R12.2, R14.2, R15.2, R16.2, R22.2, R30.2, R31.2, R32.2, R48.2, R49.2, R53.2, R54.2, RJ1.4, RJ1.5, U11.1, U12.6, U13.6, U14.6, U15.1, U16.B2, U17.5, U20.5, U21.6, U22.6, U3.6, U4.19, U4.27, U4.33, U4.39, U4.40, U4.46, U9.8
- net +5V: now also J4.1, J4.2; no longer C3.+, C38.POS, C4.1, L1.P$2, R42.2, TP2.PAD, U18.7, U19.7, U6.26, U6.8, VR1.4
- net A: now also J4.14; no longer R50.2, R51.1, U9.6
- net B: now also J4.12; no longer R49.1, R51.2, U9.7
- net EE_D+: now also J4.13; no longer U4.4
- net EE_D-: now also J4.11; no longer U4.3
- net ESTOP: now also J4.4
- net GND: now also J4.10, J4.3, J4.9; no longer C13.1, C14.1, C18.1, C19.1, C20.1, C21.1, C22.1, C23.1, C24.1, C25.1, C26.1, C3.-, C30.1, C31.1, C32.1, C33.1, C34.1, C35.1, C37.NEG, C38.NEG, C4.2, C60.1, C61.1, C73.1, C74.1, C76.1, C77.1, C78.1, C79.1, C80.1, C81.1, C82.1, C83.1, C84.1, C85.1, D2.NEG, J20.1, J20.11, J20.13, J20.15, J20.5, J20.9, J21.2, J22.4, J23.2, J3.4, J4.6, J4.GND, J4.GND2, J4.NC, LED10.C, LED12.C, LED13.C, LED14.C, LED6.C, LED7.C, R13.1, R33.2, R34.2, R35.1, R50.1, RJ1.SHLD0, RJ1.SHLD1, U11.2, U11.5, U12.2, U12.5, U13.2, U13.5, U14.2, U14.5, U15.2, U15.5, U16.C2, U16.C3, U17.3, U18.6, U19.6, U20.3, U21.2, U21.5, U22.2, U22.5, U3.2, U4.34, U4.44, U4.PAD, U9.5, VR1.3, VR1.GND
- net N$1: now also C11.2, R10.2, U6.26, U6.8; no longer C77.2
- net N$2: now also C12.2, R10.1, U6.25; no longer C78.2, FB3.1, J22.1
- net PWR1: no longer R56.2, U18.8
- net PWR2: no longer R55.2, U18.5
- net ULC_D+: now also J4.7; no longer U4.2
- net ULC_D-: now also J4.5; no longer U4.1
- net USBMCU+: now also J4.8; no longer U4.9
- net USBMCU-: now also J4.6; no longer U4.8
