File: EAGLE/EMC03 - Motion Control/EMC03-Motion Control.brd (EAGLE design)
At the start: 100 x 86.6 mm, 140 parts, among them J1 UART0, J10 S4B-PH-SM4, J11 S4B-PH-SM4, J12 S4B-PH-SM4, J13 S5B-PH-SM4, J14 S5B-PH-SM4, J15 S5B-PH-SM4, J16 S8B-PH-SM4, J17 S8B-PH-SM4, J18 S6B-PH-SM4, J19 S6B-PH-SM4, J2 FTSH-105-1-L-DV, J3 CONN-OSTTH050160, J5 S3B-PH-SM4, J6 S3B-PH-SM4, J7 S3B-PH-SM4, J9 ESTOP, Q1 12MHz, U1 LPC1768, U2 SP3485, U5 74AHCT, U6 TMC2130-LA, U7 TMC2130-LA, U8 TMC2130-LA

Commit message: Finalized schematics (minus potential LDO regulator) for all boards. Layout partially done for EFD01
Parts:
- removed C36: 220uF, TinWhiskers:C-SMD-10MM
- removed C50: 470uF, TinWhiskers:C-SMD-10MM
- removed D1: 1N4148, SparkFun-DiscreteSemi:SOD-123
- removed J16: S8B-PH-SM4, TinWhiskers:CONN-JST-PH-2.0MM-8P-SMT-RA
- removed J18: S6B-PH-SM4, TinWhiskers:CONN-JST-PH-2.0MM-6P-SMT-RA
- removed J3: CONN-OSTTH050160, FirePick:CONN-OSTTH050160
- removed J4: (no value), !con-lstb:MA07-2
- removed J9: ESTOP, TinWhiskers:CON-HDR-2POS-MALE
- removed L2: 100uH, TinWhiskers:L-SMD-12.5MM
- removed LOGO11: LOGO-FIREPICKLARGE, FirePick:LOGO-FIREPICK
- removed LOGO2: LOGO-OSHWMEDIUM, FirePick:LOGO-OSHW-MEDIUM
- removed LOGO3, LOGO7, LOGO9: LOGO-CC-BY-SALARGE, FirePick:LOGO-CC-BY-SA
- removed R27: 100K, TinWhiskers:R0603
- removed R28: 10K, TinWhiskers:R0603
- removed R29: 4.7K, TinWhiskers:R0603
- removed U5: 74AHCT, TinWhiskers:SC70
- added C13, C14, C18, C19: 4.7uF, TinWhiskers:C0603
- added C20, C21, C22: 100uF, TinWhiskers:C-SMD-6.3MM
- added C3: 220uF, TinWhiskers:C-SMD-6.3MM
- added C4: 470uF, TinWhiskers:C-SMD-6.3MM
- added L1: 100uH, TinWhiskers:2020
- added R11, R12: 2R2, TinWhiskers:R0603
- added TB1: DC-IN, TinWhiskers:TBLOCK-3-5MM-OSTTH030160
- added U3: 74LVC, TinWhiskers:SOT-23-5
- C11: value 4.7 uF -> 4.7uF
- C16, C40, C63: value 470 nF -> 470nF
- C17, C41, C42, C52, C64, C65: value 100 nF -> 100nF
- R10: value 2.2 -> 2R2; device TinWhiskers:R1206 -> TinWhiskers:R0603
- moved J17 276.4 mm to (-111.4, -154.7), turned to 0 degrees
- moved R10 129.5 mm to (-16.3, 39.8)
- moved C11 40.4 mm to (-99.4, -107.7)
- moved C12 40.4 mm to (-99.4, -112.8)
Connections:
- removed net !ENABLE_BUF: U1.38, U5.2
- removed net EE_D+: J16.7, J4.13
- removed net EE_D-: J16.8, J4.11
- removed net ESTOP_OE: D1.A, J9.2, R27.1, U5.1
- removed net PWR1: J16.6
- removed net PWR2: J17.6
- removed net ULC_D+: J17.7, J4.7
- removed net ULC_D-: J17.8, J4.5
- new net !ENABLE_LPC: U1.38, U3.2
- new net !ENABLE_MOD: J17.2, J19.2, U3.1
- new net N$3: C19.2, R11.1, U8.25
- new net N$4: C18.2, R11.2, U8.26, U8.8
- new net N$6: C13.2, R12.2, U7.26, U7.8
- net !ENABLE: now also U3.4; no longer J16.2, J17.2, J18.2, J19.2, R28.1, U5.4
- net +24V: now also C20.POS, C21.POS, C22.POS, TB1.1; no longer J16.1, J18.1
- net +3V3: now also C4.POS, L1.2, U3.5; no longer C50.POS, L2.P$2, R27.2, R28.2, U5.5
- net +5V: now also C3.POS, J17.6, TB1.2; no longer C36.POS, J18.6, J4.1, J4.2, U7.26, U7.8, U8.26, U8.8
- net A: no longer J16.4, J18.4, J4.14
- net B: no longer J16.5, J18.5, J4.12
- net ESTOP: no longer D1.C, J4.4
- net GND: now also C13.1, C14.1, C18.1, C19.1, C20.NEG, C21.NEG, C22.NEG, C3.NEG, C4.NEG, TB1.3, U3.3; no longer C36.NEG, C50.NEG, J16.3, J18.3, J4.10, J4.3, J4.9, R29.1, U5.3
- net N$16: now also L1.1; no longer L2.P$1
- net N$5: now also C14.2, R12.1, U7.25; no longer J9.1, R29.2
- net USBMCU+: now also J17.7; no longer J4.8
- net USBMCU-: now also J17.8; no longer J4.6
