File: EAGLE/EMC03 - Motion Control/EMC03-Motion Control.sch (EAGLE design)
At the start: 209 parts, among them J1 UART0, J10 S4B-PH-SM4, J11 S4B-PH-SM4, J12 S4B-PH-SM4, J13 S5B-PH-SM4, J14 S5B-PH-SM4, J15 S5B-PH-SM4, J16 S8B-PH-SM4, J17 S8B-PH-SM4, J18 S6B-PH-SM4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

Commit message: Arranged EMC03 board as much as possible. Updated PCB Checklist with testpoint data. Updated test points to pads, as per schematic instructions.
Parts:
- TP1, TP2, TP3, TP4: device FirePick:CONN-TESTPOINT -> TinWhiskers:TPAD
Changed lines of the file:
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@@
 <attribute name="PARTNO" value="S3B-PH-SM4-TB(LF)(SN)"/>
 </part>
-<part name="TP3" library="FirePick" deviceset="CONN-TESTPOINT" device="" value="+24V">
+<part name="TP3" library="TinWhiskers" deviceset="TPAD" device="" value="+24V">
 <attribute name="DNP" value="T"/>
 <attribute name="PARTNO" value="N/A"/>
 </part>
-<part name="TP4" library="FirePick" deviceset="CONN-TESTPOINT" device="" value="GND">
+<part name="TP4" library="TinWhiskers" deviceset="TPAD" device="" value="GND">
 <attribute name="DNP" value="T"/>
 <attribute name="PARTNO" value="N/A"/>
 </part>
-<part name="TP2" library="FirePick" deviceset="CONN-TESTPOINT" device="" value="+5V">
+<part name="TP2" library="TinWhiskers" deviceset="TPAD" device="" value="+5V">
 <attribute name="DNP" value="T"/>
 <attribute name="PARTNO" value="N/A"/>
 </part>
 <part name="+5V" library="supply1" deviceset="+5V" device=""/>
-<part name="TP1" library="FirePick" deviceset="CONN-TESTPOINT" device="" value="+3.3V">
+<part name="TP1" library="TinWhiskers" deviceset="TPAD" device="" value="+3.3V">
 <attribute name="DNP" value="T"/>
 <attribute name="PARTNO" value="N/A"/>
