File: EAGLE/EFD01 - Crsl. Feeder/EFD01 - C. Feeder.sch (EAGLE design)
At the start: 0 parts

Commit message: Updated schematic to integrate Intel Edison into EMC03 (USB chip for serial console, USB hub for all peripherals and associated EEPROM, second RS-485 transceiver for Edison). USB-B connection has been removed and replaced with a panel-mount version connected by vertical header. Ethernet interface connects to USB hub now, and MicroSD interfaces with Edison instead of LPC1768. Some of the 5V switching regulators have been removed for the time being. All necessary parts for EMC03 have been added to TinWhiskers library. EFD01 Schematic has a complete set of connections, could use some tidying up before layout.
Parts:
- added C1: 10nF, TinWhiskers:CPL-CAP-X7R-0603-10NF-50V
- added C2: 100nF, TinWhiskers:CPL-CAP-X7R-0603-100NF-50V
- added C3, C35, C36: 1uF, TinWhiskers:CPL-CAP-X5R-0603-1UF-50V
- added C4, C5: 12pF, TinWhiskers:CPL-CAP-C0G-0603-12PF-50V
- added C6: 0.1uF, TinWhiskers:CPL-CAP-X7R-0603-100NF-50V
- added J1: MOD TOOL, TinWhiskers:CPL-CON-JST-2.0MM-6P-M-RA
- added J2: SPI, TinWhiskers:CPL-CON-HEADER-0.1IN-6P-M
- added J3: MOT, TinWhiskers:CPL-CON-JST-2.0MM-4P-M-RA
- added J4: FTDI, TinWhiskers:CPL-CON-JST-2.0MM-6P-M-RA
- added LED1: GREEN, TinWhiskers:CPL-LED-0603-GREEN
- added Q1: BSS138, TinWhiskers:CPL-TRN-NFET-SOT23
- added Q2: 16MHz, TinWhiskers:CPL-OSC-CRY-16MHZ-18PF
- added R1: 10K, TinWhiskers:TC33X-2
- added R10: 120, TinWhiskers:CPL-RES-0603-120-0.1W
- added R11, R3, R4: 1K, TinWhiskers:CPL-RES-0603-1K-0.1W
- added R12, R9: 10K, TinWhiskers:CPL-RES-0603-10K-0.1W
- added R2: 100R, TinWhiskers:CPL-RES-0603-100-0.1W
- added R5, R6: 0R22, TinWhiskers:CPL-RES-1206-0.22-0.5W
- added R7: 20K, TinWhiskers:CPL-RES-0603-20K-0.1W
- added R8: 1M, TinWhiskers:CPL-RES-0603-1M-0.1W
- added U1: SP3485, TinWhiskers:SP3485
- added U2: TCST1030, TinWhiskers:TCSTXX30
- added U3: AT328, TinWhiskers:CPL-MCU-ATMEL-AT328-32TQFP
- added U4: DRV8825, TinWhiskers:CPL-MDR-DRV8825
- added VR1: TC1015-3.3VCT713, TinWhiskers:CPL-REG-LIN-3.3V-0.1A
Connections:
- new net !ENBL: J1.2, U3.PD5, U4.!ENBL
- new net +24V: C2.1, J1.1, U4.VMA, U4.VMB
- new net +3V3: C36.2, R3.2, U1.8, VR1.5
- new net +5V: C35.2, J1.6, J2.2, J4.3, R10.2, R11.2, R12.2, R9.2, U3.AVCC, U3.VCC@4, U3.VCC@6, U4.!RESET, U4.!SLEEP, VR1.1, VR1.3
- new net A: J1.4, R2.1, R4.2, U1.6
- new net AOUT1: J3.1, U4.AOUT1
- new net AOUT2: J3.2, U4.AOUT2
- new net B: J1.5, R2.2, R3.1, U1.7
- new net BOUT1: J3.3, U4.BOUT1
- new net BOUT2: J3.4, U4.BOUT2
- new net DI: J4.5, U1.4, U3.PD1
- new net DIR: U3.PD4, U4.DIR
- new net DTR1: U1.2, U1.3
- new net GND: C35.1, C36.1, C4.1, C5.1, J1.3, J2.6, J4.1, J4.2, Q1.S, R1.A, R4.1, R5.1, R6.1, U1.5, U2.LED_K, U2.NPN_E, U3.AREF, U3.GND@21, U3.GND@3, U3.GND@5, U3.TAB, U4.GND@14, U4.GND@28, U4.PAD
- new net MISO: J2.1, U3.PB3
- new net MOSI: J2.4, U3.PB4
- new net N$1: LED1.C, Q1.D
- new net N$13: C3.2, R7.1, U4.MODE0, U4.MODE1, U4.MODE2, U4.V3P3OUT
- new net N$14: R1.E, R7.2
- new net N$15: R1.S, U4.AVREF, U4.BVREF
- new net N$16: C6.1, J4.6
- new net N$2: R10.1, U2.LED_A
- new net N$3: LED1.A, R11.1
- new net N$5: C1.2, U4.CP1
- new net N$6: C1.1, U4.CP2
- new net N$7: C2.2, U4.VCP
- new net N$8: R5.2, U4.ISENA
- new net N$9: R6.2, U4.ISENB
- new net O_OUT: Q1.G, R9.1, U2.NPN_C, U3.PD2
- new net RESET: C6.2, J2.5, R12.1, U3.PC6
- new net RO: J4.4, U1.1, U3.PD0
- new net SCK: J2.3, U3.PB5
- new net SS: U3.PB2
- new net STEP: U3.PD3, U4.STEP
- new net XTAL1: C4.2, Q2.1, R8.1, U3.PB6
- new net XTAL2: C5.2, Q2.2, R8.2, U3.PB7
