File: EAGLE/EFD01 - Crsl. Feeder/EFD01 - C. Feeder.sch (EAGLE design)
At the start: 35 parts, among them J1 MOD TOOL, J2 SPI, J3 MOT, J4 FTDI, Q1 BSS138, Q2 16MHz, U1 SP3485, U2 TCST1030, U3 ATMEGA238, U4 DRV8825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

Commit message: BOMs complete for all FPD boards
Parts:
- J2: PARTNO (none) -> 67996-206HLF
- U$1: PARTNO (none) -> *
- U5: PARTNO (none) -> SN74LVC1G32DBVR
Changed lines of the file:
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@@
 <?xml version="1.0" encoding="utf-8"?>
 <!DOCTYPE eagle SYSTEM "eagle.dtd">
-<eagle version="7.3.0">
+<eagle version="7.4.0">
 <drawing>
 <settings>
@@
 <part name="LOGO2" library="FirePick" deviceset="LOGO-FIREPICK" device="LARGE"/>
 <part name="SUPPLY17" library="TinWhiskers" deviceset="GND" device=""/>
-<part name="U5" library="TinWhiskers" deviceset="CPL-IC-LOGIC-OR-1CH-74LVC" device="" value="74LVC"/>
+<part name="U5" library="TinWhiskers" deviceset="CPL-IC-LOGIC-OR-1CH-74LVC" device="" value="74LVC">
+<attribute name="PARTNO" value="SN74LVC1G32DBVR"/>
+</part>
 <part name="SUPPLY18" library="TinWhiskers" deviceset="GND" device=""/>
 <part name="+3V4" library="supply1" deviceset="+3V3" device=""/>
-<part name="J2" library="TinWhiskers" deviceset="CPL-CON-HEADER-0.1IN-2X3P-M" device="" value="SPI"/>
+<part name="J2" library="TinWhiskers" deviceset="CPL-CON-HEADER-0.1IN-2X3P-M" device="" value="SPI">
+<attribute name="PARTNO" value="67996-206HLF"/>
+</part>
 <part name="P+4" library="supply1" deviceset="+5V" device=""/>
 <part name="P+11" library="supply1" deviceset="+5V" device=""/>
 <part name="SUPPLY4" library="TinWhiskers" deviceset="GND" device=""/>
-<part name="U$1" library="!tin-whiskers-logo" deviceset="TIN-WHISKERS" device="SMALL"/>
+<part name="U$1" library="!tin-whiskers-logo" deviceset="TIN-WHISKERS" device="SMALL">
+<attribute name="PARTNO" value="*"/>
+</part>
 </parts>
 <sheets>
@@
 <instance part="LOGO2" gate="G$1" x="81.28" y="10.16"/>
 <instance part="SUPPLY17" gate="GND" x="350.52" y="45.72"/>
-<instance part="U5" gate="G$1" x="220.98" y="198.12"/>
+<instance part="U5" gate="G$1" x="220.98" y="198.12">
+<attribute name="PARTNO" x="220.98" y="198.12" size="1.778" layer="96" display="off"/>
+</instance>
 <instance part="SUPPLY18" gate="GND" x="205.74" y="190.5"/>
 <instance part="+3V4" gate="G$1" x="228.6" y="205.74" smashed="yes">
@@
 <instance part="J2" gate="G$1" x="134.62" y="152.4" smashed="yes" rot="R180">
 <attribute name="NAME" x="132.08" y="157.48" size="1.778" layer="125" ratio="12"/>
+<attribute name="PARTNO" x="134.62" y="152.4" size="1.778" layer="96" display="off"/>
 </instance>
 <instance part="P+4" gate="1" x="116.84" y="165.1" smashed="yes">
@@
 <attribute name="VALUE" x="147.955" y="139.065" size="1.778" layer="96"/>
 </instance>
-<instance part="U$1" gate="G$1" x="10.16" y="33.02"/>
+<instance part="U$1" gate="G$1" x="10.16" y="33.02">
+<attribute name="PARTNO" x="10.16" y="33.02" size="1.778" layer="96" display="off"/>
+</instance>
 </instances>
 <busses>
