File: EAGLE/EFD01 - Crsl. Feeder/EFD01 - C. Feeder.brd (EAGLE design)
At the start: 160 x 100 mm, 34 parts, among them J1 MOD TOOL, J2 SPI, J3 MOT, J4 FTDI, Q1 BSS138, Q2 16MHz, U1 SP3485, U2 TCST1030, U3 ATMEGA238, U4 DRV8825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

Commit message: Updated all boards to include changes for production
Parts:
- J4: device TinWhiskers:CONN-JST-PH-2.0MM-6P-SMT-RA -> TinWhiskers:CON-HDR-6POS-MALE
- U3: device TinWhiskers:32-TQFN -> TinWhiskers:32-TQF(ATMEGA)
- moved Q2 21.3 mm to (16.9, 31.2), turned to 225 degrees
- moved C5 19.8 mm to (13.1, 34.1), turned to 225 degrees
- moved R8 19.2 mm to (11.8, 31.6), turned to 135 degrees
- moved C4 18.4 mm to (14.9, 32.5), turned to 225 degrees
- moved LOGO2 16.4 mm to (2.04, 13.1)
- moved J4 0.10 mm to (42.1, 14.6), turned to 90 degrees
Connections:
- net GND: no longer U3.PAD
Routing:
- net XTAL1: track 31.1 -> 16.4 mm
- net XTAL2: track 29.1 -> 14.9 mm, vias 2 -> 0
- net GND: track 57.3 -> 46.3 mm, vias 40 -> 27
- net +5V: track 37.6 -> 31.9 mm
- net N$9: track 3.72 -> 6.51 mm, vias 0 -> 2
- net N$14: track 15.2 -> 17.8 mm
- net N$13: track 42.4 -> 44.4 mm
- net STEP: track 45.8 -> 44.1 mm, vias 4 -> 5
- net N$16: track 16.2 -> 16.8 mm, vias 2 -> 1
- net +24V: vias 0 -> 4
- added copper zone on layer 15, net +24V
Other:
- board size 160 x 100 mm -> 50 x 50 mm
- board text added: "MOD TOOL"
- board text added: "MOT"

Commit message: Final(??) Versions of FPD boards.
Parts:
- moved C1 3.52 mm to (40.8, 45.3), turned to 0 degrees
- moved C2 3.11 mm to (38.5, 43.9), turned to 270 degrees
- moved C5 2.09 mm to (11.0, 34.2)
- moved C4 2.09 mm to (12.8, 32.6)
- moved R8 2.09 mm to (9.71, 31.7)
- moved J1 1.94 mm to (16.4, 41.8)
- moved J3 1.94 mm to (31.2, 41.8)
Routing:
- net +24V: track 26.7 -> 13.1 mm, vias 4 -> 5
- net VCP: track 5.65 -> 0.00 mm
- net XTAL1: track 16.4 -> 19.0 mm
- net N$6: track 4.00 -> 6.51 mm
- net A: track 40.6 -> 38.4 mm
- net BOUT2: track 19.5 -> 17.5 mm
- net XTAL2: track 14.9 -> 16.8 mm
- net AOUT1: track 11.4 -> 9.54 mm
- net B: track 36.4 -> 34.9 mm
- net AOUT2: track 14.5 -> 12.9 mm
- net +5V: track 31.9 -> 30.5 mm
- net BOUT1: track 18.5 -> 17.2 mm
- net DIR: track 76.0 -> 77.0 mm
- net GND: track 46.3 -> 47.1 mm
- net N$5: track 5.19 -> 5.95 mm
Other:
- board text added: "U4"
