File: EAGLE/EFP01 - Front Panel Board/EFP01 - Front Panel Board.sch (EAGLE design)
At the start: 150 parts, among them J1 PWRBTN, J16 S8B-PH-SM4, J17 S8B-PH-SM4, J18 S6B-PH-SM4, J2 ESTOP, J20 Intel EDISON, J3 USB-A(2.0), J5 LCD, J6 S8B-PH-SM4, J7 USB-B, Q2 25MHz, U1 74LVC1T45, U10 FT231XS-R, U11 74LVC1T45, U12 74LVC1T45, U13 74LVC1T45, U14 74LVC1T45, U15 74LVC1T45, U17 OR, U18 MIC2026-1YM, U19 MIC2026-1YM, U2 74LVC1T45, U20 OR, U21 74LVC1T45, U22 74LVC1T45, U23 74LVC1T45, U24 74LVC1T45, U25 74LVC1T45, U26 74LVC1T45, U27 74LVC1T45, U28 74LVC1T45, U3 93LC66A, U30 74LVC1T45, U4 LAN9514, U5 74LVC1T45, U6 74LVC1T45, U7 74LVC1T45, U8 74LVC1T45, U9 SP3485

Commit message: Final(??) Versions of FPD boards.
Connections:
- net DM renamed SCON_N
- net DP renamed SCON_P
- net RXD renamed SC_N
- net RXDO renamed SCED_N
- net TXD renamed SCED_P
- net TXDO renamed SC_P
Changed lines of the file:
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@@
-</segment>
-</net>
-<net name="DP" class="0">
-<segment>
-<wire x1="165.1" y1="76.2" x2="190.5" y2="76.2" width="0.1524" layer="91"/>
-<label x="182.88" y="76.2" size="1.778" layer="95"/>
-<pinref part="J7" gate="G$1" pin="2"/>
-</segment>
-<segment>
-<wire x1="220.98" y1="66.04" x2="208.28" y2="66.04" width="0.1524" layer="91"/>
-<label x="208.28" y="66.04" size="1.778" layer="95"/>
-<pinref part="U10" gate="G$1" pin="USBDP"/>
-</segment>
-</net>
-<net name="DM" class="0">
-<segment>
-<wire x1="165.1" y1="73.66" x2="193.04" y2="73.66" width="0.1524" layer="91"/>
-<label x="182.88" y="73.66" size="1.778" layer="95"/>
-<pinref part="J7" gate="G$1" pin="3"/>
-</segment>
-<segment>
-<wire x1="220.98" y1="68.58" x2="208.28" y2="68.58" width="0.1524" layer="91"/>
-<label x="208.28" y="68.58" size="1.778" layer="95"/>
-<pinref part="U10" gate="G$1" pin="USBDM"/>
 </segment>
 </net>
@@
 </segment>
 </net>
-<net name="TXD" class="0">
-<segment>
-<pinref part="J20" gate="G$1" pin="GP135"/>
-<wire x1="365.76" y1="195.58" x2="373.38" y2="195.58" width="0.1524" layer="91"/>
-<label x="370.84" y="195.58" size="1.778" layer="95"/>
-</segment>
-<segment>
-<pinref part="U12" gate="G$1" pin="3"/>
-<wire x1="312.42" y1="121.92" x2="304.8" y2="121.92" width="0.1524" layer="91"/>
-<label x="304.8" y="121.92" size="1.778" layer="95"/>
-</segment>
-</net>
-<net name="RXD" class="0">
-<segment>
-<wire x1="246.38" y1="78.74" x2="256.54" y2="78.74" width="0.1524" layer="91"/>
-<label x="251.46" y="78.74" size="1.778" layer="95"/>
-<pinref part="U10" gate="G$1" pin="RXD"/>
-</segment>
-<segment>
-<pinref part="U11" gate="G$1" pin="3"/>
-<wire x1="350.52" y1="121.92" x2="342.9" y2="121.92" width="0.1524" layer="91"/>
-<label x="342.9" y="121.92" size="1.778" layer="95"/>
-</segment>
-</net>
 <net name="USB0_P" class="0">
 <segment>
@@
 <wire x1="327.66" y1="195.58" x2="317.5" y2="195.58" width="0.1524" layer="91"/>
 <label x="314.96" y="195.58" size="1.778" layer="95"/>
-</segment>
-</net>
-<net name="TXDO" class="0">
-<segment>
-<wire x1="246.38" y1="81.28" x2="256.54" y2="81.28" width="0.1524" layer="91"/>
-<label x="251.46" y="81.28" size="1.778" layer="95"/>
-<pinref part="U10" gate="G$1" pin="TXD"/>
-</segment>
-<segment>
-<pinref part="U12" gate="G$1" pin="4"/>
-<wire x1="332.74" y1="121.92" x2="340.36" y2="121.92" width="0.1524" layer="91"/>
-<label x="335.28" y="121.92" size="1.778" layer="95"/>
-</segment>
-</net>
-<net name="RXDO" class="0">
-<segment>
-<pinref part="J20" gate="G$1" pin="GP134"/>
-<wire x1="365.76" y1="198.12" x2="373.38" y2="198.12" width="0.1524" layer="91"/>
-<label x="370.84" y="198.12" size="1.778" layer="95"/>
-</segment>
-<segment>
-<pinref part="U11" gate="G$1" pin="4"/>
-<wire x1="370.84" y1="121.92" x2="378.46" y2="121.92" width="0.1524" layer="91"/>
-<label x="373.38" y="121.92" size="1.778" layer="95"/>
 </segment>
 </net>
@@
 </segment>
 </net>
+<net name="SCON_P" class="0">
+<segment>
+<wire x1="165.1" y1="76.2" x2="190.5" y2="76.2" width="0.1524" layer="91"/>
+<label x="182.88" y="76.2" size="1.778" layer="95"/>
+<pinref part="J7" gate="G$1" pin="2"/>
+</segment>
+<segment>
+<wire x1="220.98" y1="66.04" x2="208.28" y2="66.04" width="0.1524" layer="91"/>
+<label x="208.28" y="66.04" size="1.778" layer="95"/>
+<pinref part="U10" gate="G$1" pin="USBDP"/>
+</segment>
+</net>
+<net name="SCON_N" class="0">
+<segment>
+<wire x1="165.1" y1="73.66" x2="190.5" y2="73.66" width="0.1524" layer="91"/>
+<label x="182.88" y="73.66" size="1.778" layer="95"/>
+<pinref part="J7" gate="G$1" pin="3"/>
+</segment>
+<segment>
+<wire x1="220.98" y1="68.58" x2="208.28" y2="68.58" width="0.1524" layer="91"/>
+<label x="208.28" y="68.58" size="1.778" layer="95"/>
+<pinref part="U10" gate="G$1" pin="USBDM"/>
+</segment>
+</net>
+<net name="SCED_P" class="0">
+<segment>
+<pinref part="U12" gate="G$1" pin="3"/>
+<wire x1="312.42" y1="121.92" x2="304.8" y2="121.92" width="0.1524" layer="91"/>
+<label x="302.26" y="121.92" size="1.778" layer="95"/>
+</segment>
+<segment>
+<pinref part="J20" gate="G$1" pin="GP135"/>
+<wire x1="365.76" y1="195.58" x2="373.38" y2="195.58" width="0.1524" layer="91"/>
+<label x="370.84" y="195.58" size="1.778" layer="95"/>
+</segment>
+</net>
+<net name="SCED_N" class="0">
+<segment>
+<pinref part="U11" gate="G$1" pin="4"/>
+<wire x1="370.84" y1="121.92" x2="378.46" y2="121.92" width="0.1524" layer="91"/>
+<label x="373.38" y="121.92" size="1.778" layer="95"/>
+</segment>
+<segment>
+<pinref part="J20" gate="G$1" pin="GP134"/>
+<wire x1="365.76" y1="198.12" x2="373.38" y2="198.12" width="0.1524" layer="91"/>
+<label x="370.84" y="198.12" size="1.778" layer="95"/>
+</segment>
+</net>
+<net name="SC_N" class="0">
+<segment>
+<pinref part="U11" gate="G$1" pin="3"/>
+<wire x1="350.52" y1="121.92" x2="342.9" y2="121.92" width="0.1524" layer="91"/>
+<label x="342.9" y="121.92" size="1.778" layer="95"/>
+</segment>
+<segment>
+<wire x1="246.38" y1="78.74" x2="256.54" y2="78.74" width="0.1524" layer="91"/>
+<label x="251.46" y="78.74" size="1.778" layer="95"/>
+<pinref part="U10" gate="G$1" pin="RXD"/>
+</segment>
+</net>
+<net name="SC_P" class="0">
+<segment>
+<wire x1="246.38" y1="81.28" x2="256.54" y2="81.28" width="0.1524" layer="91"/>
+<label x="251.46" y="81.28" size="1.778" layer="95"/>
+<pinref part="U10" gate="G$1" pin="TXD"/>
+</segment>
+<segment>
+<pinref part="U12" gate="G$1" pin="4"/>
+<wire x1="332.74" y1="121.92" x2="340.36" y2="121.92" width="0.1524" layer="91"/>
+<label x="335.28" y="121.92" size="1.778" layer="95"/>
+</segment>
+</net>

Commit message: Created BOM for EFP01
Parts:
- C1, C10, C15, C16, C17, C27, C28, C29, C33, C34, C35, C36, C37, C38, C39, C40, C41, C42, C43, C44, C45, C46, C47, C48, C49, C5, C6, C7, C8, C9: PARTNO (none) -> GMK107BJ104KAHT
- C2: device TinWhiskers:CPL-CAP-X7R-0603-100NF-50V -> TinWhiskers:CPL-CAP-X5R-0603-0.1UF-35V; PARTNO UMK107B7104KA-T -> GMK107BJ104KAHT
- C3, C4: PARTNO (none) -> EMVH350ADA100MF60G
- J1: PARTNO (none) -> S4B-PH-SM4-TB(LF)(SN)
- J16, J17, J6: PARTNO S8B-PH-SM4-TB(LF)(SN) -> B8B-PH-SM4-TB(LF)(SN)
- J18: PARTNO S6B-PH-SM4-TB(LF)(SN) -> B6B-PH-SM4-TB(LF)(SN)
- J2: PARTNO (none) -> S2B-PH-SM4-TB(LF)(SN)
- J3: PARTNO (none) -> 1734085-1
- J5: PARTNO (none) -> TSW-117-07-T-D
- J7: PARTNO (none) -> 1734517-1
- R1: PARTNO (none) -> RC0603FR-074K7L
- R2: PARTNO (none) -> RC0603FR-0710KL
- R3: PARTNO (none) -> RC0603JR-070RL
- TB1: PARTNO (none) -> OSTTH030160
- U10: PARTNO * -> FT231XS-R
- U17, U20: PARTNO (none) -> SN74LVC1G32DBVR
- U21, U22, U23, U24, U5, U6: PARTNO (none) -> 74LVC1T45GW,125
- VR1: PARTNO (none) -> LMS8117AMP-3.3/NOPB
Connections:
- net +3V3: now also C2.2; no longer C2.1
- net GND: now also C2.1; no longer C2.2
