File: EAGLE/EFP01 - Front Panel Board/EFP01 - Front Panel Board.sch (EAGLE design)
At the start: 151 parts, among them J1 PWRBTN, J16 S8B-PH-SM4, J17 S8B-PH-SM4, J18 S6B-PH-SM4, J2 ESTOP, J20 Intel EDISON, J3 USB-A(2.0), J5 LCD, J6 S8B-PH-SM4, J7 USB-B, Q2 25MHz, U1 74LVC1T45, U10 FT231XS-R, U11 74LVC1T45, U12 74LVC1T45, U13 74LVC1T45, U14 74LVC1T45, U15 74LVC1T45, U17 OR, U18 MIC2026-1YM, U19 MIC2026-1YM, U2 74LVC1T45, U20 OR, U21 74LVC1T45, U22 74LVC1T45, U23 74LVC1T45, U24 74LVC1T45, U25 74LVC1T45, U26 74LVC1T45, U27 74LVC1T45, U28 74LVC1T45, U3 93LC66A, U30 74LVC1T45, U4 LAN9514, U5 74LVC1T45, U6 74LVC1T45, U7 74LVC1T45, U8 74LVC1T45, U9 SP3485

Commit message: Fixed BOM, began adding DFM changes
Connections:
- net +3V3: now also U10.VCC
Changed lines of the file:
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@@
 <pinref part="+3V22" gate="G$1" pin="+3V3"/>
 <wire x1="220.98" y1="78.74" x2="208.28" y2="78.74" width="0.1524" layer="91"/>
-<wire x1="208.28" y1="78.74" x2="208.28" y2="86.36" width="0.1524" layer="91"/>
+<wire x1="208.28" y1="78.74" x2="208.28" y2="81.28" width="0.1524" layer="91"/>
 <pinref part="U10" gate="G$1" pin="VCCIO"/>
+<pinref part="U10" gate="G$1" pin="VCC"/>
+<wire x1="208.28" y1="81.28" x2="208.28" y2="86.36" width="0.1524" layer="91"/>
+<wire x1="208.28" y1="81.28" x2="220.98" y2="81.28" width="0.1524" layer="91"/>
+<junction x="208.28" y="81.28"/>
 </segment>
 <segment>

Commit message: Routing for differential pairs included in EFP01. Minor changes to BOM, inventory list.
Parts:
- J1: device TinWhiskers:CPL-CON-JST-2.0MM-4P-M-SMT-RA -> TinWhiskers:CPL-CON-JST-2.0MM-4P-M-SMT-VRT
- J2: device TinWhiskers:CPL-CON-JST-2.0MM-2P-M-SMT-RA -> TinWhiskers:CPL-CON-JST-2.0MM-2P-M-SMT-VRT
Changed lines of the file:
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@@
 </part>
 <part name="P+4" library="supply1" deviceset="+24V" device=""/>
-<part name="J1" library="TinWhiskers" deviceset="CPL-CON-JST-2.0MM-4P-M-SMT-RA" device="" value="PWRBTN">
+<part name="J1" library="TinWhiskers" deviceset="CPL-CON-JST-2.0MM-4P-M-SMT-VRT" device="" value="PWRBTN">
 <attribute name="PARTNO" value="S4B-PH-SM4-TB(LF)(SN)"/>
 </part>
-<part name="J2" library="TinWhiskers" deviceset="CPL-CON-JST-2.0MM-2P-M-SMT-RA" device="" value="ESTOP">
+<part name="J2" library="TinWhiskers" deviceset="CPL-CON-JST-2.0MM-2P-M-SMT-VRT" device="" value="ESTOP">
 <attribute name="PARTNO" value="S2B-PH-SM4-TB(LF)(SN)"/>
 </part>
