File: EAGLE/EFP01 - Front Panel Board/EFP01 - Front Panel Board.brd (EAGLE design)
At the start: 200 x 65 mm, 150 parts, among them J1 PWRBTN, J16 S8B-PH-SM4, J17 S8B-PH-SM4, J18 S6B-PH-SM4, J2 ESTOP, J20 Intel EDISON, J3 USB-A(2.0), J5 LCD, J6 S8B-PH-SM4, J7 USB-B, Q2 25MHz, U1 74LVC1T45, U10 FT231XS-R, U11 74LVC1T45, U12 74LVC1T45, U13 74LVC1T45, U14 74LVC1T45, U15 74LVC1T45, U17 OR, U18 MIC2026-1YM, U19 MIC2026-1YM, U2 74LVC1T45, U20 OR, U21 74LVC1T45, U22 74LVC1T45, U23 74LVC1T45, U24 74LVC1T45, U25 74LVC1T45, U26 74LVC1T45, U27 74LVC1T45, U28 74LVC1T45, U3 93LC66A, U30 74LVC1T45, U4 LAN9514, U5 74LVC1T45, U6 74LVC1T45, U7 74LVC1T45, U8 74LVC1T45, U9 SP3485

Commit message: Minor changes to EFP01.  One show-stopper DRC error (overlapping traces).  Added logo and P/N.  Other misc. tweaks.  Generated Gerbers for Rev--.
Parts:
- added U$1: TIN-WHISKERSTSTOP, !tin-whiskers-logo:TIN-WHISKERS-TSTOP
Routing:
- net GND: track 346.4 -> 325.9 mm, vias 109 -> 111
- net +3V3: track 214.6 -> 217.1 mm
- net 74DIR: vias 8 -> 10
Other:
- board text added: "EFP01 Rev --"
