File: EAGLE/ECAM02 - EE2.0/ECAM02-EE2.0.sch (EAGLE design)
At the start: 61 parts, among them J1 MODULAR TOOL, J2 SPI, J3 MOT, J4 FTDI, J5 S4B-PH-SM4, J6 SOL+PUMP, J7 RINGLIGHT, Q2 16MHz, U1 SP3485, U10 MCP4725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

Commit message: BOMs finished, inventory sheet created.
Parts:
- R2: value 100R -> 120R; device TinWhiskers:CPL-RES-0603-100-0.1W -> TinWhiskers:CPL-RES-0603-120-0.1W; PARTNO RC0603FR-07100RL -> RC0603FR-07120RL
Changed lines of the file:
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@@
 <part name="P+1" library="supply1" deviceset="+24V" device=""/>
 <part name="P+2" library="supply1" deviceset="+5V" device=""/>
-<part name="R2" library="TinWhiskers" deviceset="CPL-RES-0603-100-0.1W" device="" value="100R">
-<attribute name="PARTNO" value="RC0603FR-07100RL"/>
+<part name="R2" library="TinWhiskers" deviceset="CPL-RES-0603-120-0.1W" device="" value="120R">
+<attribute name="PARTNO" value="RC0603FR-07120RL"/>
 </part>
 <part name="R3" library="TinWhiskers" deviceset="CPL-RES-0603-1K-0.1W" device="" value="1K">

Commit message: Updated some of the attributes on schematics which contained incorrect part numbers. Similarly adjusted BOMs and inventory/PO form to reflect these changes.
Parts:
- J3: PARTNO S4B-PH-SM4-TB(LF)(SN) -> B4B-PH-K-S(LF)(SN)
- X1: PARTNO MPXV5004GP -> MPXV5100DP
Changed lines of the file:
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@@
 <part name="SUPPLY8" library="TinWhiskers" deviceset="GND" device=""/>
 <part name="J3" library="TinWhiskers" deviceset="CPL-CON-JST-2.0MM-4P-M-THRU-VRT" device="" value="MOT">
-<attribute name="PARTNO" value="S4B-PH-SM4-TB(LF)(SN)"/>
+<attribute name="PARTNO" value="B4B-PH-K-S(LF)(SN)"/>
 </part>
 <part name="SUPPLY13" library="TinWhiskers" deviceset="GND" device=""/>
@@
 </part>
 <part name="X1" library="TinWhiskers" deviceset="CPL-SEN-PRS-MPXV5100DP" device="" value="MPXV5100DP">
-<attribute name="PARTNO" value="MPXV5004GP"/>
+<attribute name="PARTNO" value="MPXV5100DP"/>
 </part>
 <part name="C9" library="TinWhiskers" deviceset="CPL-CAP-X5R-0603-1UF-50V" device="" value="1uF">
